File: rocket-logger-basic.brd (EAGLE design)
At the start: 58.5 x 62 mm, 61 parts, among them IC1 CC430F513X, Q2 MOSFET-PCHANNEL, U2 MAX1555, U3 MCP73831, X1 0896BM15A0001, X2 USB-MICROB, X3 SMA-142-0701-801/806

Commit message: basic logger done
Parts:
- removed JP1: (no value), SparkFun:S2B-PH
- moved R4 10.3 mm to (9.05, 22.3)
- moved C26 3.23 mm to (8.43, 25.5), turned to 270 degrees
- moved C11 0.41 mm to (7.18, 25.4)
- moved R13 0.25 mm to (10.3, 22.3)
- moved R5 0.20 mm to (2.80, 20.5)
- moved C12 0.20 mm to (7.81, 22.3)
- moved LED3 0.20 mm to (9.96, 28.9)
- moved C1 0.15 mm to (10.2, 19.4)
- moved R7 0.15 mm to (3.39, 18.6)
- moved C17 0.10 mm to (2.06, 18.7)
Connections:
- net GND: no longer JP1.1
- net N$2: no longer JP1.2
- net N$25: now also R4.2
Routing:
- net N$25: track 4.15 -> 9.93 mm
- net GND: track 71.5 -> 74.5 mm, vias 17 -> 35
- net N$2: track 28.3 -> 27.2 mm
- net N$18: track 8.66 -> 9.28 mm
Other:
- board text added: "Jan 14"
- board text added: "Matt Brejza"
- board text added: "Rocket Altimeter"

Commit message: finishing off, almost done
Other:
- outline, holes or cut-outs redrawn
- board text added: "Rev. 1"
- board text removed: "untent and label"
Changed lines of the file:
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@@
 <layer number="21" name="tPlace" color="16" fill="1" visible="yes" active="yes"/>
 <layer number="22" name="bPlace" color="14" fill="1" visible="yes" active="yes"/>
-<layer number="23" name="tOrigins" color="15" fill="1" visible="no" active="yes"/>
+<layer number="23" name="tOrigins" color="15" fill="1" visible="yes" active="yes"/>
 <layer number="24" name="bOrigins" color="15" fill="1" visible="yes" active="yes"/>
 <layer number="25" name="tNames" color="7" fill="1" visible="no" active="yes"/>
@@
 <layer number="116" name="Patch_BOT" color="9" fill="4" visible="no" active="yes"/>
 <layer number="121" name="_tsilk" color="7" fill="1" visible="no" active="yes"/>
-<layer number="122" name="_bsilk" color="7" fill="1" visible="yes" active="yes"/>
+<layer number="122" name="_bsilk" color="7" fill="1" visible="no" active="yes"/>
 <layer number="125" name="_tNames" color="7" fill="1" visible="no" active="yes"/>
 <layer number="144" name="Drill_legend" color="7" fill="1" visible="no" active="yes"/>
@@
 <wire x1="0" y1="0" x2="19.75" y2="0" width="0" layer="20"/>
 <wire x1="17" y1="5.5" x2="17" y2="27.6344" width="0" layer="20"/>
-<wire x1="17" y1="27.6344" x2="17" y2="33.1208" width="0" layer="20"/>
-<wire x1="17" y1="33.1208" x2="17" y2="44.5" width="0" layer="20"/>
 <wire x1="19.75" y1="50" x2="1.75" y2="50" width="0" layer="20"/>
 <hole x="2.5" y="47.75" drill="3"/>
-<rectangle x1="21.75" y1="32.5" x2="23.655" y2="47.74" layer="1" rot="R180"/>
 <rectangle x1="24.2638" y1="14.4244" x2="41.4088" y2="37.2844" layer="16"/>
 <text x="10.25" y="37.75" size="1.016" layer="122" ratio="12" rot="MR270">ON</text>
 <text x="8.5" y="37.75" size="1.016" layer="122" ratio="12" rot="MR270">ACT</text>
-<wire x1="0" y1="48.25" x2="0" y2="23.368" width="0" layer="20"/>
 <wire x1="0" y1="23.368" x2="0" y2="0" width="0" layer="20"/>
 <wire x1="22.5" y1="2.75" x2="19.75" y2="0" width="0" layer="20" curve="-90"/>
@@
 <wire x1="19.75" y1="44.5" x2="17" y2="44.5" width="0" layer="20"/>
 <wire x1="0" y1="48.25" x2="1.75" y2="50" width="0" layer="20" curve="-90"/>
-<hole x="17" y="45.25" drill="0.381"/>
-<hole x="17" y="46" drill="0.381"/>
-<hole x="17" y="46.75" drill="0.381"/>
-<hole x="17" y="47.5" drill="0.381"/>
-<hole x="17" y="48.25" drill="0.381"/>
-<hole x="17" y="49" drill="0.381"/>
-<hole x="17" y="49.5" drill="0.381"/>
+<hole x="17.2032" y="45.0468" drill="0.381"/>
+<hole x="17.2032" y="45.7968" drill="0.381"/>
+<hole x="17.2032" y="46.5468" drill="0.381"/>
+<hole x="17.2032" y="47.2968" drill="0.381"/>
+<hole x="17.2032" y="48.0468" drill="0.381"/>
+<hole x="17.2032" y="48.7968" drill="0.381"/>
+<hole x="17.2032" y="49.5" drill="0.381"/>
 <hole x="17" y="5" drill="0.381"/>
 <hole x="17" y="4.25" drill="0.381"/>
@@
 <wire x1="19.75" y1="50" x2="22.5" y2="47.25" width="0" layer="20" curve="-90"/>
 <circle x="2.4384" y="47.752" radius="2.649403125" width="0.2032" layer="1"/>
-<text x="-1.8288" y="13.208" size="1.778" layer="1" rot="R90">untent and label</text>
-<hole x="3.6504" y="35.0588" drill="3"/>
-<wire x1="2.6416" y1="37.1856" x2="4.4704" y2="37.1856" width="0" layer="20"/>
-<wire x1="4.4704" y1="37.1856" x2="6.096" y2="35.7632" width="0" layer="20" curve="-90"/>
-<wire x1="6.096" y1="35.7632" x2="6.096" y2="33.9344" width="0" layer="20"/>
+<hole x="3.6504" y="35.262" drill="3"/>
+<wire x1="2.6416" y1="37.3888" x2="4.4704" y2="37.3888" width="0" layer="20"/>
+<wire x1="4.4704" y1="37.3888" x2="6.096" y2="35.9664" width="0" layer="20" curve="-90"/>
+<wire x1="6.096" y1="35.9664" x2="6.096" y2="33.9344" width="0" layer="20"/>
 <wire x1="6.096" y1="33.9344" x2="6.9088" y2="33.1216" width="0" layer="20" curve="90"/>
 <wire x1="6.9088" y1="33.1216" x2="17.0688" y2="33.1216" width="0" layer="20"/>
 <hole x="5.824" y="33.2612" drill="0.381"/>
-<hole x="4.808" y="33.2612" drill="0.381"/>
-<hole x="3.9952" y="33.2612" drill="0.381"/>
-<hole x="2.9792" y="33.2612" drill="0.381"/>
-<hole x="2.1664" y="33.2612" drill="0.381"/>
-<hole x="1.3536" y="33.2612" drill="0.381"/>
+<hole x="5.0112" y="33.2612" drill="0.381"/>
+<hole x="4.1984" y="33.2612" drill="0.381"/>
+<hole x="3.3856" y="33.2612" drill="0.381"/>
+<hole x="2.5728" y="33.2612" drill="0.381"/>
+<hole x="1.76" y="33.2612" drill="0.381"/>
 <wire x1="19.75" y1="33.1208" x2="17" y2="33.1208" width="0" layer="20"/>
 <wire x1="19.75" y1="33.1344" x2="22.5" y2="30.3844" width="0" layer="20" curve="-90"/>
@@
 <wire x1="19.75" y1="27.6344" x2="17" y2="27.6344" width="0" layer="20"/>
 <hole x="19.7032" y="30.3844" drill="3"/>
-<hole x="16.7968" y="32.6344" drill="0.381"/>
+<hole x="16.7968" y="32.8376" drill="0.381"/>
+<hole x="16.7968" y="32.228" drill="0.381"/>
 <hole x="16.7968" y="31.4152" drill="0.381"/>
-<hole x="16.7968" y="32.0248" drill="0.381"/>
-<hole x="16.7968" y="30.8056" drill="0.381"/>
-<hole x="16.7968" y="29.9928" drill="0.381"/>
-<hole x="16.7968" y="29.18" drill="0.381"/>
-<hole x="16.7968" y="28.3672" drill="0.381"/>
-<hole x="16.7968" y="27.7576" drill="0.381"/>
+<hole x="16.7968" y="30.6024" drill="0.381"/>
+<hole x="16.7968" y="29.7896" drill="0.381"/>
+<hole x="16.7968" y="28.9768" drill="0.381"/>
+<hole x="16.7968" y="28.164" drill="0.381"/>
 <dimension x1="0" y1="0" x2="0" y2="33.1216" x3="-20.7264" y3="16.5608" layer="107"/>
 <dimension x1="0" y1="0" x2="17.0688" y2="0" x3="8.5344" y3="-15.6464" layer="107"/>
-<rectangle x1="17.4752" y1="33.6296" x2="21.9964" y2="39.624" layer="1" rot="R180"/>
 <dimension x1="0" y1="0" x2="0" y2="37.1856" x3="-27.2288" y3="18.5928" layer="107"/>
 <wire x1="1.2192" y1="24.384" x2="0.8128" y2="23.9776" width="0" layer="20" curve="-90"/>
 <wire x1="0.8128" y1="23.9776" x2="0.6096" y2="23.9776" width="0" layer="20"/>
 <wire x1="0.6096" y1="23.9776" x2="0" y2="23.368" width="0" layer="20" curve="90"/>
-<wire x1="1.2192" y1="24.384" x2="1.2192" y2="35.7632" width="0" layer="20"/>
-<wire x1="1.2192" y1="35.7632" x2="2.6416" y2="37.1856" width="0" layer="20" curve="-90"/>
+<wire x1="1.2192" y1="24.384" x2="1.2192" y2="35.9664" width="0" layer="20"/>
+<wire x1="1.2192" y1="35.9664" x2="2.6416" y2="37.3888" width="0" layer="20" curve="-90"/>
 <rectangle x1="-7.5184" y1="-20.9804" x2="0" y2="0" layer="1"/>
-<rectangle x1="11.2776" y1="34.6964" x2="13.8176" y2="37.7952" layer="1"/>
-<rectangle x1="8.5344" y1="33.6804" x2="9.3472" y2="35.4076" layer="1" rot="R90"/>
 <text x="8.5344" y="31.6992" size="1.016" layer="122" font="vector" ratio="20" rot="MR180">CHG</text>
 <text x="13.4112" y="31.6992" size="1.016" layer="122" font="vector" ratio="20" rot="MR180">PWR</text>
@@
 <text x="2.7686" y="16.2052" size="0.8128" layer="122" font="vector" ratio="16" rot="SMR270">Jan 14</text>
 <text x="12.9286" y="19.6088" size="0.8128" layer="122" font="vector" ratio="16" rot="SMR270">Rocket Altimeter</text>
+<text x="4" y="16.2" size="0.8128" layer="122" font="vector" ratio="16" rot="SMR270">Rev. 1</text>
 </plain>
 <attributes>
@@
 <wire x1="15.8496" y1="22.352" x2="15.8496" y2="22.1488" width="0.2032" layer="16"/>
 <polygon width="0.2032" layer="16">
-<vertex x="1.016" y="34.544"/>
-<vertex x="16.6624" y="34.7472"/>
-<vertex x="17.0688" y="34.3408"/>
+<vertex x="1.016" y="33.3248"/>
+<vertex x="16.4592" y="33.3248"/>
+<vertex x="16.8656" y="32.9184"/>
 <vertex x="17.0688" y="0.6096"/>
 <vertex x="16.4592" y="0"/>
 <vertex x="0.4064" y="0"/>
 <vertex x="0" y="0.4064"/>
-<vertex x="0" y="34.1376"/>
+<vertex x="0.2032" y="32.512"/>
 </polygon>
 <wire x1="2.0516" y1="9.5248" x2="2.0516" y2="9.1636" width="0.2032" layer="1"/>

Commit message: added part values
Parts:
- R1: value (none) -> 56k2
- R10, R4: value (none) -> 100k
- R11: value (none) -> 330
- R13: value (none) -> 17k
- R5, R6, R7: value (none) -> 4k7
- R8, R9: value (none) -> 2M
Changed lines of the file:
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@@
 <?xml version="1.0" encoding="utf-8"?>
 <!DOCTYPE eagle SYSTEM "eagle.dtd">
-<eagle version="6.2">
+<eagle version="6.5.0">
 <drawing>
 <settings>
@@
 <hole x="16.7968" y="28.9768" drill="0.381"/>
 <hole x="16.7968" y="28.164" drill="0.381"/>
-<dimension x1="0" y1="0" x2="0" y2="33.1216" x3="-20.7264" y3="16.5608" layer="107"/>
-<dimension x1="0" y1="0" x2="17.0688" y2="0" x3="8.5344" y3="-15.6464" layer="107"/>
-<dimension x1="0" y1="0" x2="0" y2="37.1856" x3="-27.2288" y3="18.5928" layer="107"/>
+<dimension x1="0" y1="0" x2="0" y2="33.1216" x3="-20.7264" y3="16.5608" textsize="3.5" layer="107"/>
+<dimension x1="0" y1="0" x2="17.0688" y2="0" x3="8.5344" y3="-15.6464" textsize="3.5" layer="107"/>
+<dimension x1="0" y1="0" x2="0" y2="37.1856" x3="-27.2288" y3="18.5928" textsize="3.5" layer="107"/>
 <wire x1="1.2192" y1="24.384" x2="0.8128" y2="23.9776" width="0" layer="20" curve="-90"/>
 <wire x1="0.8128" y1="23.9776" x2="0.6096" y2="23.9776" width="0" layer="20"/>
@@
 </class>
 </classes>
-<designrules>
+<designrules name="default">
 <description language="de">&lt;b&gt;EAGLE Design Rules&lt;/b&gt;
 &lt;p&gt;
@@
 <element name="C13" library="resistor" package="C0402" value="" x="1.8436" y="7.9468"/>
 <element name="C14" library="resistor" package="C0402" value="" x="2.5" y="0.7968"/>
-<element name="R1" library="rcl" package="R0402" value="" x="11.5" y="7.5468" rot="R90"/>
+<element name="R1" library="rcl" package="R0402" value="56k2" x="11.5" y="7.5468" rot="R90"/>
 <element name="X3" library="con-coax" package="J502-ND-142-0701-801/806" value="SMA-142-0701-801/806" x="10.5" y="0" rot="R90">
 <attribute name="OC_NEWARK" value="90F2624" x="10.5" y="0" size="1.778" layer="27" rot="R90" display="off"/>
@@
 <element name="C16" library="resistor" package="C0402" value="100n" x="3.2512" y="10.25" rot="R90"/>
 <element name="C17" library="resistor" package="C0402" value="" x="2.0644" y="18.6624" rot="R270"/>
-<element name="R4" library="rcl" package="R0402" value="" x="9.0456" y="22.266" rot="R90"/>
+<element name="R4" library="rcl" package="R0402" value="100k" x="9.0456" y="22.266" rot="R90"/>
 <element name="S2" library="SparkFun" package="TACTILE_SWITCH_SMD" value="SWITCH-MOMENTARY-2SMD" x="5.1264" y="29.368" rot="MR180"/>
 <element name="JP2" library="SparkFun" package="1X02" value="" x="14.9824" y="21.096" rot="R180"/>
-<element name="R6" library="rcl" package="R0402" value="" x="4.5412" y="18.6444" rot="R90"/>
-<element name="R7" library="rcl" package="R0402" value="" x="3.3864" y="18.6444" rot="R90"/>
+<element name="R6" library="rcl" package="R0402" value="4k7" x="4.5412" y="18.6444" rot="R90"/>
+<element name="R7" library="rcl" package="R0402" value="4k7" x="3.3864" y="18.6444" rot="R90"/>
 <element name="D3" library="diode" package="SOD523" value="" x="2.7192" y="22.5396" rot="R180"/>
 <element name="D4" library="diode" package="SOD523" value="" x="2.6872" y="21.5236"/>
-<element name="R5" library="rcl" package="R0402" value="" x="2.8048" y="20.5276" rot="R180"/>
+<element name="R5" library="rcl" package="R0402" value="4k7" x="2.8048" y="20.5276" rot="R180"/>
 <element name="SG1" library="buzzer" package="EFBRD24C411" value="EFBRD24C411" x="0.25" y="-51">
 <attribute name="OC_NEWARK" value="unknown" x="0.25" y="-51" size="1.016" layer="27" ratio="12" display="off"/>
@@
 <attribute name="TP_SIGNAL_NAME" value="" x="1.4224" y="1.6256" size="1.778" layer="28" rot="MR0" display="off"/>
 </element>
-<element name="R8" library="rcl" package="R0402" value="" x="15.24" y="25.6032"/>
-<element name="R9" library="rcl" package="R0402" value="" x="15.24" y="23.1648" rot="R180"/>
+<element name="R8" library="rcl" package="R0402" value="2M" x="15.24" y="25.6032"/>
+<element name="R9" library="rcl" package="R0402" value="2M" x="15.24" y="23.1648" rot="R180"/>
 <element name="C27" library="resistor" package="C0402" value="" x="15.24" y="24.384" rot="R180"/>
-<element name="R10" library="rcl" package="R0402" value="" x="16.2052" y="6.5024" rot="R90"/>
+<element name="R10" library="rcl" package="R0402" value="100k" x="16.2052" y="6.5024" rot="R90"/>
 <element name="C18" library="resistor" package="C0402" value="" x="15.0876" y="6.5024" rot="R90"/>
 <element name="JP3" library="SparkFun" package="1X04" value="" x="14.986" y="18.034" rot="R270"/>
-<element name="R11" library="rcl" package="R0402" value="" x="7.9756" y="28.194" rot="R270"/>
+<element name="R11" library="rcl" package="R0402" value="330" x="7.9756" y="28.194" rot="R270"/>
 <element name="LED3" library="SparkFun" package="LED-0603" value="" x="9.9568" y="28.8544" rot="MR180"/>
 <element name="U2" library="SparkFun" package="SOT23-5" value="MAX1555" x="-28.0416" y="-60.96"/>
@@
 <attribute name="PROD_ID" value="IC-09995" x="11.176" y="24.7904" size="1.778" layer="27" rot="R90" display="off"/>
 </element>
-<element name="R13" library="rcl" package="R0402" value="" x="10.2608" y="22.2504" rot="R270"/>
+<element name="R13" library="rcl" package="R0402" value="17k" x="10.2608" y="22.2504" rot="R270"/>
 <element name="C19" library="resistor" package="C0402" value="" x="7.62" y="19.3548" rot="R270"/>
 </elements>

Commit message: updating component values
Parts:
- removed D1: (no value), diode:SOD523
- removed IC3: (no value), SparkFun:SOT23-5
- removed Q2: MOSFET-PCHANNEL, SparkFun:SOT23
- removed R12: (no value), rcl:R0402
- removed U2: MAX1555, SparkFun:SOT23-5
- C1: value (none) -> 470n
- C10, C11, C12, C19, C26, C3, C5: value (none) -> 1u
- C13, C14: value (none) -> 27p
- C17, C2, C4, C6, C9: value (none) -> 100n
- C18: value (none) -> 2n2
- C8: value (none) -> 100p
- R2, R3: value (none) -> 110
Connections:
- removed net N$20: D1.C, IC3.1, Q2.3
- removed net N$21: D1.A, Q2.1, R12.1, U2.1
- removed net N$22: R12.2
- removed net N$27: Q2.2, U2.5
Changed lines of the file:
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@@
 <element name="LED2" library="SparkFun" package="LED-0603" value="" x="15.396" y="28.8728" rot="MR0"/>
 <element name="IC2" library="SparkFun" package="SOT23-5" value="" x="5.4348" y="22.3068" rot="R180"/>
-<element name="C1" library="resistor" package="C0402" value="" x="10.162" y="19.3636" rot="R270"/>
-<element name="C2" library="resistor" package="C0402" value="" x="8.8636" y="19.3636" rot="R270"/>
-<element name="C3" library="resistor" package="C0402" value="" x="0.8632" y="10.1748" rot="R90"/>
-<element name="C4" library="resistor" package="C0402" value="" x="0.8684" y="18.6428" rot="R270"/>
-<element name="C5" library="resistor" package="C0402" value="" x="13.8984" y="6.5348" rot="R90"/>
-<element name="C6" library="resistor" package="C0402" value="" x="12.6484" y="7.5468" rot="R90"/>
+<element name="C1" library="resistor" package="C0402" value="470n" x="10.162" y="19.3636" rot="R270"/>
+<element name="C2" library="resistor" package="C0402" value="100n" x="8.8636" y="19.3636" rot="R270"/>
+<element name="C3" library="resistor" package="C0402" value="1u" x="0.8632" y="10.1748" rot="R90"/>
+<element name="C4" library="resistor" package="C0402" value="100n" x="0.8684" y="18.6428" rot="R270"/>
+<element name="C5" library="resistor" package="C0402" value="1u" x="13.8984" y="6.5348" rot="R90"/>
+<element name="C6" library="resistor" package="C0402" value="100n" x="12.6484" y="7.5468" rot="R90"/>
 <element name="C7" library="resistor" package="C0402" value="" x="18.9076" y="7.7032" rot="R90"/>
-<element name="C8" library="resistor" package="C0402" value="" x="6" y="8.2968"/>
-<element name="C9" library="resistor" package="C0402" value="" x="6" y="7.1484"/>
-<element name="C10" library="resistor" package="C0402" value="" x="6" y="6"/>
+<element name="C8" library="resistor" package="C0402" value="100p" x="6" y="8.2968"/>
+<element name="C9" library="resistor" package="C0402" value="100n" x="6" y="7.1484"/>
+<element name="C10" library="resistor" package="C0402" value="1u" x="6" y="6"/>
 <element name="X2" library="SparkFun" package="USB-MICROB" value="USB-MICROB" x="2.7032" y="28.1048" rot="R270"/>
-<element name="C11" library="resistor" package="C0402" value="" x="7.1832" y="25.4304" rot="R90"/>
-<element name="C12" library="resistor" package="C0402" value="" x="7.8064" y="22.2652" rot="R90"/>
+<element name="C11" library="resistor" package="C0402" value="1u" x="7.1832" y="25.4304" rot="R90"/>
+<element name="C12" library="resistor" package="C0402" value="1u" x="7.8064" y="22.2652" rot="R90"/>
 <element name="Q1" library="SparkFun" package="CRYSTAL-SMD-5X3" value="" x="2.25" y="4.2968" rot="R90"/>
-<element name="C13" library="resistor" package="C0402" value="" x="1.8436" y="7.9468"/>
-<element name="C14" library="resistor" package="C0402" value="" x="2.5" y="0.7968"/>
+<element name="C13" library="resistor" package="C0402" value="27p" x="1.8436" y="7.9468"/>
+<element name="C14" library="resistor" package="C0402" value="27p" x="2.5" y="0.7968"/>
 <element name="R1" library="rcl" package="R0402" value="56k2" x="11.5" y="7.5468" rot="R90"/>
 <element name="X3" library="con-coax" package="J502-ND-142-0701-801/806" value="SMA-142-0701-801/806" x="10.5" y="0" rot="R90">
@@
 <attribute name="OC_FARNELL" value="1608592" x="10.5" y="0" size="1.778" layer="27" rot="R90" display="off"/>
 </element>
-<element name="R2" library="rcl" package="R0402" value="" x="7.974" y="30.6648" rot="R90"/>
-<element name="R3" library="rcl" package="R0402" value="" x="6.778" y="30.6508" rot="R270"/>
+<element name="R2" library="rcl" package="R0402" value="110" x="7.974" y="30.6648" rot="R90"/>
+<element name="R3" library="rcl" package="R0402" value="110" x="6.778" y="30.6508" rot="R270"/>
 <element name="C15" library="resistor" package="C0402" value="10u" x="2.0516" y="10.1748" rot="R90"/>
 <element name="C16" library="resistor" package="C0402" value="100n" x="3.2512" y="10.25" rot="R90"/>
-<element name="C17" library="resistor" package="C0402" value="" x="2.0644" y="18.6624" rot="R270"/>
+<element name="C17" library="resistor" package="C0402" value="100n" x="2.0644" y="18.6624" rot="R270"/>
 <element name="R4" library="rcl" package="R0402" value="100k" x="9.0456" y="22.266" rot="R90"/>
 <element name="S2" library="SparkFun" package="TACTILE_SWITCH_SMD" value="SWITCH-MOMENTARY-2SMD" x="5.1264" y="29.368" rot="MR180"/>
@@
 <attribute name="OC_FARNELL" value="unknown" x="0.25" y="-51" size="1.016" layer="27" ratio="12" display="off"/>
 </element>
-<element name="C26" library="resistor" package="C0402" value="" x="8.4328" y="25.4516" rot="R270"/>
+<element name="C26" library="resistor" package="C0402" value="1u" x="8.4328" y="25.4516" rot="R270"/>
 <element name="L1" library="wuerth-elektronik" package="0603" value="" x="15.24" y="8.4836"/>
 <element name="TP1" library="testpad" package="B1,27" value="PTR1B1,27" x="1.4224" y="4.064" rot="MR0">
@@
 <element name="C27" library="resistor" package="C0402" value="" x="15.24" y="24.384" rot="R180"/>
 <element name="R10" library="rcl" package="R0402" value="100k" x="16.2052" y="6.5024" rot="R90"/>
-<element name="C18" library="resistor" package="C0402" value="" x="15.0876" y="6.5024" rot="R90"/>
+<element name="C18" library="resistor" package="C0402" value="2n2" x="15.0876" y="6.5024" rot="R90"/>
 <element name="JP3" library="SparkFun" package="1X04" value="" x="14.986" y="18.034" rot="R270"/>
 <element name="R11" library="rcl" package="R0402" value="330" x="7.9756" y="28.194" rot="R270"/>
 <element name="LED3" library="SparkFun" package="LED-0603" value="" x="9.9568" y="28.8544" rot="MR180"/>
-<element name="U2" library="SparkFun" package="SOT23-5" value="MAX1555" x="-28.0416" y="-60.96"/>
-<element name="IC3" library="SparkFun" package="SOT23-5" value="" x="-31.0896" y="-60.96"/>
-<element name="D1" library="diode" package="SOD523" value="" x="-31.2928" y="-65.4304"/>
-<element name="Q2" library="SparkFun" package="SOT23" value="MOSFET-PCHANNEL" x="-34.3408" y="-64.4144"/>
-<element name="R12" library="rcl" package="R0402" value="" x="-34.3408" y="-68.8848"/>
 <element name="U$1" library="Mine" package="JST-ZR-2" value="JST-ZR-2" x="12.0904" y="28.448"/>
 <element name="U$2" library="Mine" package="JST-ZR-2-SMD" value="JST-ZR-2SMD" x="12.192" y="28.7528"/>
@@
 </element>
 <element name="R13" library="rcl" package="R0402" value="17k" x="10.2608" y="22.2504" rot="R270"/>
-<element name="C19" library="resistor" package="C0402" value="" x="7.62" y="19.3548" rot="R270"/>
+<element name="C19" library="resistor" package="C0402" value="1u" x="7.62" y="19.3548" rot="R270"/>
 </elements>
 <signals>
@@
 <wire x1="9.194" y1="25.45" x2="7.8136" y2="25.45" width="0.2032" layer="1"/>
 </signal>
-<signal name="N$20">
-<contactref element="D1" pad="C"/>
-<contactref element="IC3" pad="1"/>
-<contactref element="Q2" pad="3"/>
-<wire x1="-32.0396" y1="-62.2601" x2="-31.8928" y2="-65.4304" width="0" layer="19" extent="1-1"/>
-<wire x1="-34.3408" y1="-63.3144" x2="-32.0396" y2="-62.2601" width="0" layer="19" extent="1-1"/>
-</signal>
-<signal name="N$21">
-<contactref element="Q2" pad="1"/>
-<contactref element="R12" pad="1"/>
-<contactref element="U2" pad="1"/>
-<contactref element="D1" pad="A"/>
-<wire x1="-35.2908" y1="-65.5144" x2="-34.9908" y2="-68.8848" width="0" layer="19" extent="1-1"/>
-<wire x1="-30.5928" y1="-65.4304" x2="-35.2908" y2="-65.5144" width="0" layer="19" extent="1-1"/>
-<wire x1="-28.9916" y1="-62.2601" x2="-30.5928" y2="-65.4304" width="0" layer="19" extent="1-1"/>
-</signal>
-<signal name="N$22">
-<contactref element="R12" pad="2"/>
-</signal>
-<signal name="N$27">
-<contactref element="U2" pad="5"/>
-<contactref element="Q2" pad="2"/>
-<wire x1="-28.9916" y1="-59.6599" x2="-33.3908" y2="-65.5144" width="0" layer="19" extent="1-1"/>
-</signal>
 <signal name="N$1">

Commit message: changing value
Parts:
- C26: value 1u -> 4u7
Changed lines of the file:
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@@
 <attribute name="OC_FARNELL" value="unknown" x="0.25" y="-51" size="1.016" layer="27" ratio="12" display="off"/>
 </element>
-<element name="C26" library="resistor" package="C0402" value="1u" x="8.4328" y="25.4516" rot="R270"/>
+<element name="C26" library="resistor" package="C0402" value="4u7" x="8.4328" y="25.4516" rot="R270"/>
 <element name="L1" library="wuerth-elektronik" package="0603" value="" x="15.24" y="8.4836"/>
 <element name="TP1" library="testpad" package="B1,27" value="PTR1B1,27" x="1.4224" y="4.064" rot="MR0">
