File: rocket-logger.sch (EAGLE design)
At the start: 63 parts, among them IC1 CC430F513X, U1 MAX1555, X1 0896BM15A0001, X2 USB-MICROB, X3 SMA-142-0701-801/806

Commit message: some routing - changed to smaller flash
Parts:
- added C28: (no value), resistor:C-EUC0402
- added R10: (no value), rcl:R-EU_R0402
- U$6: value SPI_FLASH-X25XXSMD1 -> SPI_FLASH-X25XXSMD; device SparkFun:SPI_FLASH-X25XXSMD1 -> SparkFun:SPI_FLASH-X25XXSMD
Connections:
- net +3V3: now also R10.2
- net GND: now also C28.1
- net N$26: now also C28.2, R10.1
Other:
- note added: "check pinout"
Changed lines of the file:
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@@
 <part name="R5" library="rcl" deviceset="R-EU_" device="R0402"/>
 <part name="U$5" library="SparkFun" deviceset="SPI_FLASH-X25XX" device="SMD"/>
-<part name="U$6" library="SparkFun" deviceset="SPI_FLASH-X25XX" device="SMD1"/>
+<part name="U$6" library="SparkFun" deviceset="SPI_FLASH-X25XX" device="SMD"/>
 <part name="SG1" library="buzzer" deviceset="EFB?" device="RD24C411"/>
 <part name="S4" library="SparkFun" deviceset="SWITCH-MOMENTARY-2" device="SMD"/>
@@
 <part name="GND50" library="SparkFun" deviceset="GND" device=""/>
 <part name="GND51" library="SparkFun" deviceset="GND" device=""/>
+<part name="C28" library="resistor" deviceset="C-EU" device="C0402"/>
+<part name="R10" library="rcl" deviceset="R-EU_" device="R0402"/>
+<part name="GND52" library="supply1" deviceset="GND" device=""/>
+<part name="+3V13" library="supply1" deviceset="+3V3" device=""/>
 </parts>
 <sheets>
@@
 <text x="259.08" y="219.71" size="1.778" layer="91" rot="R90">connect -&gt; ?</text>
 <text x="111.76" y="142.24" size="1.778" layer="91" rot="R90">change to tri colour</text>
+<text x="171.45" y="115.57" size="1.778" layer="91">check pinout</text>
 </plain>
 <instances>
@@
 <instance part="GND50" gate="1" x="218.44" y="218.44" smashed="yes" rot="R270"/>
 <instance part="GND51" gate="1" x="218.44" y="49.53" smashed="yes" rot="R270"/>
+<instance part="C28" gate="G$1" x="-10.16" y="110.49" rot="MR180"/>
+<instance part="R10" gate="G$1" x="-10.16" y="125.73" rot="R90"/>
+<instance part="GND52" gate="1" x="-10.16" y="105.41"/>
+<instance part="+3V13" gate="G$1" x="-10.16" y="133.35"/>
 </instances>
 <busses>
@@
 <pinref part="GND51" gate="1" pin="GND"/>
 </segment>
+<segment>
+<pinref part="C28" gate="G$1" pin="1"/>
+<pinref part="GND52" gate="1" pin="GND"/>
+</segment>
 </net>
 <net name="N$1" class="0">
@@
 <pinref part="+3V12" gate="G$1" pin="+3V3"/>
 </segment>
+<segment>
+<pinref part="R10" gate="G$1" pin="2"/>
+<pinref part="+3V13" gate="G$1" pin="+3V3"/>
+</segment>
 </net>
 <net name="N$3" class="0">
@@
 <segment>
 <pinref part="IC1" gate="G$1" pin="RST"/>
-<wire x1="-15.24" y1="115.57" x2="-2.54" y2="115.57" width="0.1524" layer="91"/>
+<wire x1="-15.24" y1="115.57" x2="-10.16" y2="115.57" width="0.1524" layer="91"/>
+<wire x1="-10.16" y1="115.57" x2="-2.54" y2="115.57" width="0.1524" layer="91"/>
 <wire x1="-2.54" y1="115.57" x2="-2.54" y2="114.3" width="0.1524" layer="91"/>
 <pinref part="SV1" gate="1" pin="3"/>
-</segment>
-</net>
+<pinref part="C28" gate="G$1" pin="2"/>
+<junction x="-10.16" y="115.57"/>
+<pinref part="R10" gate="G$1" pin="1"/>
+<wire x1="-10.16" y1="120.65" x2="-10.16" y2="115.57" width="0.1524" layer="91"/>
+</segment>
+</net>

Commit message: adding more leds
Parts:
- added LED3, LED4: (no value), SparkFun:LED0603
- added R11, R12: (no value), rcl:R-EU_R0402
Connections:
- new net N$18: LED3.C, R12.2
- new net N$21: LED4.C, R11.2
- net +3V3: now also LED3.A, LED4.A
- net N$16: now also R12.1
- net N$17: now also R11.1
Changed lines of the file:
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@@
 <?xml version="1.0" encoding="utf-8"?>
 <!DOCTYPE eagle SYSTEM "eagle.dtd">
-<eagle version="6.2">
+<eagle version="6.4">
 <drawing>
 <settings>
@@
 <part name="GND52" library="supply1" deviceset="GND" device=""/>
 <part name="+3V13" library="supply1" deviceset="+3V3" device=""/>
+<part name="LED3" library="SparkFun" deviceset="LED" device="0603"/>
+<part name="+3V14" library="supply1" deviceset="+3V3" device=""/>
+<part name="LED4" library="SparkFun" deviceset="LED" device="0603"/>
+<part name="+3V15" library="supply1" deviceset="+3V3" device=""/>
+<part name="R11" library="rcl" deviceset="R-EU_" device="R0402"/>
+<part name="R12" library="rcl" deviceset="R-EU_" device="R0402"/>
 </parts>
 <sheets>
@@
 <instance part="GND52" gate="1" x="-10.16" y="105.41"/>
 <instance part="+3V13" gate="G$1" x="-10.16" y="133.35"/>
+<instance part="LED3" gate="G$1" x="102.87" y="153.67" rot="R270"/>
+<instance part="+3V14" gate="G$1" x="109.22" y="153.67" rot="R270"/>
+<instance part="LED4" gate="G$1" x="102.87" y="142.24" rot="R270"/>
+<instance part="+3V15" gate="G$1" x="109.22" y="142.24" rot="R270"/>
+<instance part="R11" gate="G$1" x="92.71" y="142.24"/>
+<instance part="R12" gate="G$1" x="92.71" y="153.67"/>
 </instances>
 <busses>
@@
 <pinref part="+3V13" gate="G$1" pin="+3V3"/>
 </segment>
+<segment>
+<pinref part="+3V14" gate="G$1" pin="+3V3"/>
+<pinref part="LED3" gate="G$1" pin="A"/>
+<wire x1="106.68" y1="153.67" x2="105.41" y2="153.67" width="0.1524" layer="91"/>
+</segment>
+<segment>
+<pinref part="+3V15" gate="G$1" pin="+3V3"/>
+<pinref part="LED4" gate="G$1" pin="A"/>
+<wire x1="106.68" y1="142.24" x2="105.41" y2="142.24" width="0.1524" layer="91"/>
+</segment>
 </net>
 <net name="N$3" class="0">
@@
 <wire x1="80.01" y1="149.86" x2="87.63" y2="149.86" width="0.1524" layer="91"/>
 <pinref part="R2" gate="G$1" pin="1"/>
+<pinref part="R12" gate="G$1" pin="1"/>
+<wire x1="87.63" y1="153.67" x2="87.63" y2="149.86" width="0.1524" layer="91"/>
+<junction x="87.63" y="149.86"/>
 </segment>
 </net>
@@
 <wire x1="87.63" y1="146.05" x2="82.55" y2="146.05" width="0.1524" layer="91"/>
 <wire x1="82.55" y1="146.05" x2="80.01" y2="143.51" width="0.1524" layer="91"/>
+<pinref part="R11" gate="G$1" pin="1"/>
+<wire x1="87.63" y1="142.24" x2="87.63" y2="146.05" width="0.1524" layer="91"/>
+<junction x="87.63" y="146.05"/>
 </segment>
 </net>
@@
 </segment>
 </net>
-<net name="N$9" class="0">
-<segment>
-<pinref part="R2" gate="G$1" pin="2"/>
-<pinref part="LED1" gate="G$1" pin="A"/>
-</segment>
-</net>
-<net name="N$10" class="0">
-<segment>
-<pinref part="R3" gate="G$1" pin="2"/>
-<pinref part="LED2" gate="G$1" pin="A"/>
-</segment>
-</net>
 <net name="N$28" class="0">
 <segment>
@@
 </segment>
 </net>
+<net name="N$18" class="0">
+<segment>
+<pinref part="LED3" gate="G$1" pin="C"/>
+<pinref part="R12" gate="G$1" pin="2"/>
+</segment>
+</net>
+<net name="N$20" class="0">
+<segment>
+<pinref part="R3" gate="G$1" pin="2"/>
+<pinref part="LED2" gate="G$1" pin="A"/>
+</segment>
+</net>
+<net name="N$21" class="0">
+<segment>
+<pinref part="LED4" gate="G$1" pin="C"/>
+<pinref part="R11" gate="G$1" pin="2"/>
+</segment>
+</net>
+<net name="N$9" class="0">
+<segment>
+<pinref part="R2" gate="G$1" pin="2"/>
+<pinref part="LED1" gate="G$1" pin="A"/>
+</segment>
+</net>

Commit message: removed accel from simple verison, done some routing on main one
Parts:
- removed SV1: (no value), con-lstb:MA04-1
- added JP3: (no value), SparkFun:M04PTH
Connections:
- net +3V3: now also JP3.1
- net CS_F: now also IC1.P1.7; no longer IC1.P2.0
- net GND: now also JP3.2
- net HOLD: now also IC1.P2.0; no longer IC1.P1.7
- net KEEPON: now also IC1.P1.6; no longer IC1.P2.4
- net MISO: now also IC1.P1.2; no longer IC1.P3.7
- net N$23: now also JP3.4; no longer SV1.4
- net N$26: now also JP3.3; no longer SV1.3
- net SCL: now also IC1.P3.7; no longer IC1.P1.2
- net SDA: now also IC1.P3.6; no longer IC1.P1.3
- net VBAT: now also IC1.P2.4
Changed lines of the file:
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@@
 <?xml version="1.0" encoding="utf-8"?>
 <!DOCTYPE eagle SYSTEM "eagle.dtd">
-<eagle version="6.4">
+<eagle version="6.2">
 <drawing>
 <settings>
@@
 <part name="X3" library="con-coax" deviceset="SMA-" device="142-0701-801/806"/>
 <part name="GND22" library="supply1" deviceset="GND" device=""/>
-<part name="SV1" library="con-lstb" deviceset="MA04-1" device=""/>
 <part name="R2" library="rcl" deviceset="R-EU_" device="R0402"/>
 <part name="R3" library="rcl" deviceset="R-EU_" device="R0402"/>
@@
 <part name="R11" library="rcl" deviceset="R-EU_" device="R0402"/>
 <part name="R12" library="rcl" deviceset="R-EU_" device="R0402"/>
+<part name="GND53" library="supply1" deviceset="GND" device=""/>
+<part name="+3V16" library="supply1" deviceset="+3V3" device=""/>
+<part name="JP3" library="SparkFun" deviceset="M04" device="PTH"/>
 </parts>
 <sheets>
@@
 <instance part="X3" gate="G1" x="-49.53" y="172.72"/>
 <instance part="GND22" gate="1" x="-46.99" y="167.64"/>
-<instance part="SV1" gate="1" x="-22.86" y="115.57"/>
 <instance part="R2" gate="G$1" x="92.71" y="149.86"/>
 <instance part="R3" gate="G$1" x="92.71" y="146.05"/>
@@
 <instance part="R11" gate="G$1" x="92.71" y="142.24"/>
 <instance part="R12" gate="G$1" x="92.71" y="153.67"/>
+<instance part="GND53" gate="1" x="-12.7" y="113.03" rot="R90"/>
+<instance part="+3V16" gate="G$1" x="-12.7" y="110.49" rot="R270"/>
+<instance part="JP3" gate="G$1" x="-20.32" y="113.03"/>
 </instances>
 <busses>
@@
 <pinref part="GND52" gate="1" pin="GND"/>
 </segment>
+<segment>
+<pinref part="GND53" gate="1" pin="GND"/>
+<pinref part="JP3" gate="G$1" pin="2"/>
+</segment>
 </net>
 <net name="N$1" class="0">
@@
 <wire x1="106.68" y1="142.24" x2="105.41" y2="142.24" width="0.1524" layer="91"/>
 </segment>
+<segment>
+<pinref part="+3V16" gate="G$1" pin="+3V3"/>
+<pinref part="JP3" gate="G$1" pin="1"/>
+</segment>
 </net>
 <net name="N$3" class="0">
@@
 </segment>
 <segment>
-<pinref part="IC1" gate="G$1" pin="P1.3"/>
-<wire x1="66.04" y1="167.64" x2="72.39" y2="167.64" width="0.1524" layer="91"/>
 <label x="71.12" y="167.64" size="1.778" layer="95"/>
+<wire x1="69.85" y1="167.64" x2="72.39" y2="167.64" width="0.1524" layer="91"/>
+<wire x1="69.85" y1="167.64" x2="69.85" y2="166.37" width="0.1524" layer="91"/>
 </segment>
 <segment>
@@
 <label x="172.72" y="152.4" size="1.778" layer="95"/>
 </segment>
+<segment>
+<pinref part="IC1" gate="G$1" pin="P3.6"/>
+<wire x1="66.04" y1="114.3" x2="68.58" y2="114.3" width="0.1524" layer="91"/>
+<label x="67.31" y="114.3" size="1.778" layer="95"/>
+</segment>
 </net>
 <net name="SCL" class="0">
@@
 <wire x1="223.52" y1="57.15" x2="215.9" y2="57.15" width="0.1524" layer="91"/>
 <label x="215.9" y="57.15" size="1.778" layer="95"/>
-</segment>
-<segment>
-<pinref part="IC1" gate="G$1" pin="P1.2"/>
-<wire x1="66.04" y1="170.18" x2="72.39" y2="170.18" width="0.1524" layer="91"/>
-<label x="71.12" y="170.18" size="1.778" layer="95"/>
 </segment>
 <segment>
@@
 <label x="172.72" y="149.86" size="1.778" layer="95"/>
 </segment>
+<segment>
+<pinref part="IC1" gate="G$1" pin="P3.7"/>
+<wire x1="68.58" y1="111.76" x2="66.04" y2="111.76" width="0.1524" layer="91"/>
+<label x="67.31" y="111.76" size="1.778" layer="95"/>
+</segment>
 </net>
 <net name="KEEPON" class="0">
@@
 </segment>
 <segment>
-<label x="72.39" y="142.24" size="1.778" layer="95"/>
-<pinref part="IC1" gate="G$1" pin="P2.4"/>
-<wire x1="66.04" y1="142.24" x2="74.93" y2="142.24" width="0.1524" layer="91"/>
+<pinref part="IC1" gate="G$1" pin="P1.6"/>
+<wire x1="66.04" y1="160.02" x2="77.47" y2="160.02" width="0.1524" layer="91"/>
+<label x="71.12" y="160.02" size="1.778" layer="95"/>
 </segment>
 </net>
@@
 <net name="MISO" class="0">
 <segment>
-<pinref part="IC1" gate="G$1" pin="P3.7"/>
-<wire x1="68.58" y1="111.76" x2="66.04" y2="111.76" width="0.1524" layer="91"/>
-<wire x1="66.04" y1="111.76" x2="74.93" y2="111.76" width="0.1524" layer="91"/>
 <label x="69.85" y="111.76" size="1.778" layer="95"/>
+<wire x1="69.85" y1="111.76" x2="74.93" y2="111.76" width="0.1524" layer="91"/>
+<wire x1="69.85" y1="111.76" x2="69.85" y2="110.49" width="0.1524" layer="91"/>
 </segment>
 <segment>
@@
 <label x="149.86" y="128.27" size="1.778" layer="95"/>
 </segment>
+<segment>
+<pinref part="IC1" gate="G$1" pin="P1.2"/>
+<wire x1="66.04" y1="170.18" x2="68.58" y2="170.18" width="0.1524" layer="91"/>
+<label x="67.31" y="170.18" size="1.778" layer="95"/>
+</segment>
 </net>
 <net name="MOSI" class="0">
 <segment>
 <pinref part="IC1" gate="G$1" pin="P1.1"/>
-<wire x1="66.04" y1="172.72" x2="72.39" y2="172.72" width="0.1524" layer="91"/>
+<wire x1="66.04" y1="172.72" x2="69.85" y2="172.72" width="0.1524" layer="91"/>
 <label x="72.39" y="172.72" size="1.778" layer="95"/>
+<wire x1="69.85" y1="172.72" x2="72.39" y2="172.72" width="0.1524" layer="91"/>
+<wire x1="69.85" y1="172.72" x2="69.85" y2="171.45" width="0.1524" layer="91"/>
 </segment>
 <segment>
@@
 <segment>
 <pinref part="IC1" gate="G$1" pin="P1.0"/>
-<wire x1="66.04" y1="175.26" x2="72.39" y2="175.26" width="0.1524" layer="91"/>
+<wire x1="66.04" y1="175.26" x2="69.85" y2="175.26" width="0.1524" layer="91"/>
 <label x="72.39" y="175.26" size="1.778" layer="95"/>
+<wire x1="69.85" y1="175.26" x2="72.39" y2="175.26" width="0.1524" layer="91"/>
+<wire x1="69.85" y1="175.26" x2="69.85" y2="173.99" width="0.1524" layer="91"/>
 </segment>
 <segment>
@@
 <segment>
 <pinref part="IC1" gate="G$1" pin="P1.4"/>
-<wire x1="66.04" y1="165.1" x2="74.93" y2="165.1" width="0.1524" layer="91"/>
+<wire x1="66.04" y1="165.1" x2="69.85" y2="165.1" width="0.1524" layer="91"/>
 <label x="72.39" y="165.1" size="1.778" layer="95"/>
+<wire x1="69.85" y1="165.1" x2="74.93" y2="165.1" width="0.1524" layer="91"/>
+<wire x1="69.85" y1="165.1" x2="69.85" y2="163.83" width="0.1524" layer="91"/>
 </segment>
 <segment>
@@
 </segment>
 <segment>
-<pinref part="IC1" gate="G$1" pin="P2.0"/>
-<wire x1="66.04" y1="152.4" x2="71.12" y2="152.4" width="0.1524" layer="91"/>
-<label x="71.12" y="152.4" size="1.778" layer="95"/>
+<pinref part="IC1" gate="G$1" pin="P1.7"/>
+<label x="66.04" y="157.48" size="1.778" layer="95"/>
+<wire x1="66.04" y1="157.48" x2="67.31" y2="157.48" width="0.1524" layer="91"/>
 </segment>
 </net>
@@
 </segment>
 <segment>
-<pinref part="IC1" gate="G$1" pin="P1.7"/>
-<wire x1="66.04" y1="157.48" x2="72.39" y2="157.48" width="0.1524" layer="91"/>
 <label x="71.12" y="157.48" size="1.778" layer="95"/>
+<pinref part="IC1" gate="G$1" pin="P2.0"/>
+<label x="66.04" y="152.4" size="1.778" layer="95"/>
+<wire x1="66.04" y1="152.4" x2="67.31" y2="152.4" width="0.1524" layer="91"/>
 </segment>
 </net>
@@
 <segment>
 <pinref part="IC1" gate="G$1" pin="TEST"/>
-<wire x1="-2.54" y1="119.38" x2="-7.62" y2="119.38" width="0.1524" layer="91"/>
-<pinref part="SV1" gate="1" pin="4"/>
-<wire x1="-15.24" y1="118.11" x2="-7.62" y2="118.11" width="0.1524" layer="91"/>
-<wire x1="-7.62" y1="118.11" x2="-7.62" y2="119.38" width="0.1524" layer="91"/>
+<wire x1="-2.54" y1="119.38" x2="-3.81" y2="118.11" width="0.1524" layer="91"/>
+<wire x1="-15.24" y1="118.11" x2="-3.81" y2="118.11" width="0.1524" layer="91"/>
+<pinref part="JP3" gate="G$1" pin="4"/>
 </segment>
 </net>
@@
 <pinref part="IC1" gate="G$1" pin="RST"/>
 <wire x1="-15.24" y1="115.57" x2="-10.16" y2="115.57" width="0.1524" layer="91"/>
-<wire x1="-10.16" y1="115.57" x2="-2.54" y2="115.57" width="0.1524" layer="91"/>
-<wire x1="-2.54" y1="115.57" x2="-2.54" y2="114.3" width="0.1524" layer="91"/>
-<pinref part="SV1" gate="1" pin="3"/>
+<wire x1="-10.16" y1="115.57" x2="-3.81" y2="115.57" width="0.1524" layer="91"/>
+<wire x1="-3.81" y1="115.57" x2="-2.54" y2="114.3" width="0.1524" layer="91"/>
 <pinref part="C28" gate="G$1" pin="2"/>
 <junction x="-10.16" y="115.57"/>
 <pinref part="R10" gate="G$1" pin="1"/>
 <wire x1="-10.16" y1="120.65" x2="-10.16" y2="115.57" width="0.1524" layer="91"/>
+<pinref part="JP3" gate="G$1" pin="3"/>
 </segment>
 </net>
@@
 <wire x1="68.58" y1="161.29" x2="73.66" y2="161.29" width="0.1524" layer="91"/>
 <wire x1="73.66" y1="161.29" x2="83.82" y2="171.45" width="0.1524" layer="91"/>
+<label x="68.58" y="149.86" size="1.778" layer="95"/>
 </segment>
 </net>
@@
 <label x="128.27" y="195.58" size="1.778" layer="95"/>
 </segment>
-</net>
+<segment>
+<pinref part="IC1" gate="G$1" pin="P2.4"/>
+<wire x1="66.04" y1="142.24" x2="73.66" y2="142.24" width="0.1524" layer="91"/>
+<label x="71.12" y="142.24" size="1.778" layer="95"/>
+</segment>
+</net>

Commit message: added charging led
Parts:
- added LED5: (no value), SparkFun:LED0603
- added R13: (no value), rcl:R-EU_R0402
Connections:
- new net N$10: R13.1, U1.CHG
- new net N$18: LED5.C, R13.2
- net N$1: now also LED5.A
Changed lines of the file:
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@@
 <part name="+3V16" library="supply1" deviceset="+3V3" device=""/>
 <part name="JP3" library="SparkFun" deviceset="M04" device="PTH"/>
+<part name="LED5" library="SparkFun" deviceset="LED" device="0603"/>
+<part name="R13" library="rcl" deviceset="R-EU_" device="R0402"/>
 </parts>
 <sheets>
@@
 <instance part="+3V16" gate="G$1" x="-12.7" y="110.49" rot="R270"/>
 <instance part="JP3" gate="G$1" x="-20.32" y="113.03"/>
+<instance part="LED5" gate="G$1" x="109.22" y="208.28" rot="R180"/>
+<instance part="R13" gate="G$1" x="109.22" y="218.44" rot="R270"/>
 </instances>
 <busses>
@@
 <segment>
 <pinref part="X2" gate="G$1" pin="VBUS"/>
-<wire x1="99.06" y1="227.33" x2="105.41" y2="227.33" width="0.1524" layer="91"/>
+<wire x1="99.06" y1="227.33" x2="102.87" y2="227.33" width="0.1524" layer="91"/>
+<wire x1="102.87" y1="227.33" x2="105.41" y2="227.33" width="0.1524" layer="91"/>
 <wire x1="105.41" y1="227.33" x2="105.41" y2="228.6" width="0.1524" layer="91"/>
 <pinref part="U1" gate="G$1" pin="USB"/>
@@
 <pinref part="C11" gate="G$1" pin="2"/>
 <junction x="105.41" y="228.6"/>
+<pinref part="LED5" gate="G$1" pin="A"/>
+<wire x1="109.22" y1="205.74" x2="102.87" y2="205.74" width="0.1524" layer="91"/>
+<wire x1="102.87" y1="205.74" x2="102.87" y2="227.33" width="0.1524" layer="91"/>
+<junction x="102.87" y="227.33"/>
 </segment>
 </net>
@@
 </segment>
 <segment>
-<label x="71.12" y="167.64" size="1.778" layer="95"/>
-<wire x1="69.85" y1="167.64" x2="72.39" y2="167.64" width="0.1524" layer="91"/>
-<wire x1="69.85" y1="167.64" x2="69.85" y2="166.37" width="0.1524" layer="91"/>
-</segment>
-<segment>
 <pinref part="U$1" gate="G$1" pin="SDA_SDI"/>
 <wire x1="223.52" y1="220.98" x2="214.63" y2="220.98" width="0.1524" layer="91"/>
@@
 <segment>
 <pinref part="IC1" gate="G$1" pin="P1.1"/>
-<wire x1="66.04" y1="172.72" x2="69.85" y2="172.72" width="0.1524" layer="91"/>
+<wire x1="66.04" y1="172.72" x2="72.39" y2="172.72" width="0.1524" layer="91"/>
 <label x="72.39" y="172.72" size="1.778" layer="95"/>
-<wire x1="69.85" y1="172.72" x2="72.39" y2="172.72" width="0.1524" layer="91"/>
-<wire x1="69.85" y1="172.72" x2="69.85" y2="171.45" width="0.1524" layer="91"/>
 </segment>
 <segment>
@@
 <segment>
 <pinref part="IC1" gate="G$1" pin="P1.0"/>
-<wire x1="66.04" y1="175.26" x2="69.85" y2="175.26" width="0.1524" layer="91"/>
+<wire x1="66.04" y1="175.26" x2="72.39" y2="175.26" width="0.1524" layer="91"/>
 <label x="72.39" y="175.26" size="1.778" layer="95"/>
-<wire x1="69.85" y1="175.26" x2="72.39" y2="175.26" width="0.1524" layer="91"/>
-<wire x1="69.85" y1="175.26" x2="69.85" y2="173.99" width="0.1524" layer="91"/>
 </segment>
 <segment>
@@
 <segment>
 <pinref part="IC1" gate="G$1" pin="P1.4"/>
-<wire x1="66.04" y1="165.1" x2="69.85" y2="165.1" width="0.1524" layer="91"/>
 <label x="72.39" y="165.1" size="1.778" layer="95"/>
-<wire x1="69.85" y1="165.1" x2="74.93" y2="165.1" width="0.1524" layer="91"/>
-<wire x1="69.85" y1="165.1" x2="69.85" y2="163.83" width="0.1524" layer="91"/>
+<wire x1="66.04" y1="165.1" x2="74.93" y2="165.1" width="0.1524" layer="91"/>
 </segment>
 <segment>
@@
 <label x="66.04" y="157.48" size="1.778" layer="95"/>
 <wire x1="66.04" y1="157.48" x2="67.31" y2="157.48" width="0.1524" layer="91"/>
+<wire x1="66.04" y1="157.48" x2="76.2" y2="157.48" width="0.1524" layer="91"/>
 </segment>
 </net>
@@
 </segment>
 </net>
-<net name="N$18" class="0">
+<net name="N$20" class="0">
+<segment>
+<pinref part="R3" gate="G$1" pin="2"/>
+<pinref part="LED2" gate="G$1" pin="A"/>
+</segment>
+</net>
+<net name="N$21" class="0">
+<segment>
+<pinref part="LED4" gate="G$1" pin="C"/>
+<pinref part="R11" gate="G$1" pin="2"/>
+</segment>
+</net>
+<net name="N$9" class="0">
+<segment>
+<pinref part="R2" gate="G$1" pin="2"/>
+<pinref part="LED1" gate="G$1" pin="A"/>
+</segment>
+</net>
+<net name="N$22" class="0">
 <segment>
 <pinref part="LED3" gate="G$1" pin="C"/>
@@
 </segment>
 </net>
-<net name="N$20" class="0">
-<segment>
-<pinref part="R3" gate="G$1" pin="2"/>
-<pinref part="LED2" gate="G$1" pin="A"/>
-</segment>
-</net>
-<net name="N$21" class="0">
-<segment>
-<pinref part="LED4" gate="G$1" pin="C"/>
-<pinref part="R11" gate="G$1" pin="2"/>
-</segment>
-</net>
-<net name="N$9" class="0">
-<segment>
-<pinref part="R2" gate="G$1" pin="2"/>
-<pinref part="LED1" gate="G$1" pin="A"/>
-</segment>
-</net>
+<net name="N$10" class="0">
+<segment>
+<pinref part="U1" gate="G$1" pin="CHG"/>
+<pinref part="R13" gate="G$1" pin="1"/>
+</segment>
+</net>
+<net name="N$18" class="0">
+<segment>
+<pinref part="R13" gate="G$1" pin="2"/>
+<pinref part="LED5" gate="G$1" pin="C"/>
+</segment>
+</net>
