File: rocket-logger.sch (EAGLE design)
At the start: 71 parts, among them IC1 CC430F513X, U1 MAX1555, X1 0896BM15A0001, X2 USB-MICROB, X3 SMA-142-0701-801/806

Commit message: added diodes on power path
Parts:
- added C29: (no value), resistor:C-EUC0402
- added D2, D5: (no value), diode:DIODE-SOD523
- added RN1: (no value), resistor-dil:4R-N0402ARV341
Connections:
- new net N$30: C29.2, D2.C, D5.C, IC2.IN
- net GND: now also C29.1
- net N$1: now also D5.A
- net N$2: now also D2.A; no longer IC2.IN
Other:
- moved on the sheet: C12, IC2
Changed lines of the file:
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@@
 <part name="LED5" library="SparkFun" deviceset="LED" device="0603"/>
 <part name="R13" library="rcl" deviceset="R-EU_" device="R0402"/>
+<part name="D2" library="diode" deviceset="DIODE-" device="SOD523"/>
+<part name="D5" library="diode" deviceset="DIODE-" device="SOD523"/>
+<part name="C29" library="resistor" deviceset="C-EU" device="C0402"/>
+<part name="GND54" library="SparkFun" deviceset="GND" device=""/>
+<part name="RN1" library="resistor-dil" deviceset="4R-N" device="0402ARV341"/>
 </parts>
 <sheets>
@@
 <instance part="LED1" gate="G$1" x="100.33" y="149.86" rot="R90"/>
 <instance part="LED2" gate="G$1" x="100.33" y="146.05" rot="R90"/>
-<instance part="IC2" gate="G$1" x="165.1" y="220.98"/>
+<instance part="IC2" gate="G$1" x="168.91" y="220.98"/>
 <instance part="C1" gate="G$1" x="48.26" y="195.58" rot="R270"/>
 <instance part="C2" gate="G$1" x="40.64" y="208.28" rot="MR0"/>
@@
 <instance part="GND14" gate="1" x="105.41" y="238.76" smashed="yes" rot="R180"/>
 <instance part="GND15" gate="1" x="147.32" y="233.68" smashed="yes"/>
-<instance part="GND16" gate="1" x="177.8" y="218.44" smashed="yes" rot="R90"/>
-<instance part="+3V1" gate="G$1" x="186.69" y="228.6" rot="R270"/>
-<instance part="C12" gate="G$1" x="179.07" y="234.95" rot="MR0"/>
-<instance part="GND17" gate="1" x="179.07" y="240.03" smashed="yes" rot="R180"/>
+<instance part="GND16" gate="1" x="181.61" y="218.44" smashed="yes" rot="R90"/>
+<instance part="+3V1" gate="G$1" x="189.23" y="228.6" rot="R270"/>
+<instance part="C12" gate="G$1" x="182.88" y="234.95" rot="MR0"/>
+<instance part="GND17" gate="1" x="182.88" y="240.03" smashed="yes" rot="R180"/>
 <instance part="Q1" gate="G$1" x="-6.35" y="161.29" rot="R90"/>
 <instance part="C13" gate="G$1" x="-16.51" y="163.83" rot="MR270"/>
@@
 <instance part="LED5" gate="G$1" x="109.22" y="208.28" rot="R180"/>
 <instance part="R13" gate="G$1" x="109.22" y="218.44" rot="R270"/>
+<instance part="D2" gate="G$1" x="152.4" y="228.6"/>
+<instance part="D5" gate="G$1" x="156.21" y="233.68" rot="R270"/>
+<instance part="C29" gate="G$1" x="161.29" y="234.95" rot="MR0"/>
+<instance part="GND54" gate="1" x="161.29" y="240.03" smashed="yes" rot="R180"/>
+<instance part="RN1" gate="A" x="281.94" y="76.2"/>
+<instance part="RN1" gate="B" x="281.94" y="71.12"/>
+<instance part="RN1" gate="C" x="281.94" y="66.04"/>
+<instance part="RN1" gate="D" x="281.94" y="60.96"/>
 </instances>
 <busses>
@@
 <pinref part="JP3" gate="G$1" pin="2"/>
 </segment>
+<segment>
+<pinref part="C29" gate="G$1" pin="1"/>
+<pinref part="GND54" gate="1" pin="GND"/>
+</segment>
 </net>
 <net name="N$1" class="0">
@@
 <wire x1="102.87" y1="205.74" x2="102.87" y2="227.33" width="0.1524" layer="91"/>
 <junction x="102.87" y="227.33"/>
+<pinref part="D5" gate="G$1" pin="A"/>
+<wire x1="156.21" y1="236.22" x2="156.21" y2="254" width="0.1524" layer="91"/>
+<wire x1="156.21" y1="254" x2="109.22" y2="254" width="0.1524" layer="91"/>
+<wire x1="109.22" y1="254" x2="109.22" y2="228.6" width="0.1524" layer="91"/>
+<junction x="109.22" y="228.6"/>
 </segment>
 </net>
@@
 <wire x1="139.7" y1="228.6" x2="149.86" y2="228.6" width="0.1524" layer="91"/>
 <wire x1="149.86" y1="236.22" x2="149.86" y2="228.6" width="0.1524" layer="91"/>
-<wire x1="149.86" y1="228.6" x2="157.48" y2="228.6" width="0.1524" layer="91"/>
-<junction x="149.86" y="228.6"/>
-<pinref part="IC2" gate="G$1" pin="IN"/>
 <pinref part="S1" gate="G$1" pin="1"/>
 <wire x1="139.7" y1="209.55" x2="139.7" y2="214.63" width="0.1524" layer="91"/>
@@
 <wire x1="139.7" y1="204.47" x2="139.7" y2="209.55" width="0.1524" layer="91"/>
 <junction x="139.7" y="209.55"/>
+<pinref part="D2" gate="G$1" pin="A"/>
+<junction x="149.86" y="228.6"/>
 </segment>
 </net>
@@
 <pinref part="IC2" gate="G$1" pin="OUT"/>
 <pinref part="+3V1" gate="G$1" pin="+3V3"/>
-<wire x1="175.26" y1="228.6" x2="179.07" y2="228.6" width="0.1524" layer="91"/>
+<wire x1="179.07" y1="228.6" x2="182.88" y2="228.6" width="0.1524" layer="91"/>
 <pinref part="C12" gate="G$1" pin="2"/>
-<wire x1="179.07" y1="228.6" x2="184.15" y2="228.6" width="0.1524" layer="91"/>
-<wire x1="179.07" y1="229.87" x2="179.07" y2="228.6" width="0.1524" layer="91"/>
-<junction x="179.07" y="228.6"/>
+<wire x1="182.88" y1="228.6" x2="186.69" y2="228.6" width="0.1524" layer="91"/>
+<wire x1="182.88" y1="229.87" x2="182.88" y2="228.6" width="0.1524" layer="91"/>
+<junction x="182.88" y="228.6"/>
 </segment>
 <segment>
@@
 <junction x="157.48" y="209.55"/>
 <pinref part="D4" gate="G$1" pin="C"/>
-<wire x1="157.48" y1="209.55" x2="157.48" y2="214.63" width="0.1524" layer="91"/>
-<wire x1="157.48" y1="214.63" x2="154.94" y2="214.63" width="0.1524" layer="91"/>
 <pinref part="IC2" gate="G$1" pin="EN"/>
-<wire x1="157.48" y1="223.52" x2="154.94" y2="223.52" width="0.1524" layer="91"/>
-<wire x1="154.94" y1="214.63" x2="154.94" y2="223.52" width="0.1524" layer="91"/>
+<wire x1="161.29" y1="223.52" x2="157.48" y2="223.52" width="0.1524" layer="91"/>
+<wire x1="157.48" y1="209.55" x2="157.48" y2="223.52" width="0.1524" layer="91"/>
 </segment>
 </net>
@@
 </segment>
 </net>
+<net name="N$30" class="0">
+<segment>
+<pinref part="D2" gate="G$1" pin="C"/>
+<pinref part="D5" gate="G$1" pin="C"/>
+<wire x1="154.94" y1="228.6" x2="156.21" y2="228.6" width="0.1524" layer="91"/>
+<wire x1="156.21" y1="228.6" x2="161.29" y2="228.6" width="0.1524" layer="91"/>
+<pinref part="IC2" gate="G$1" pin="IN"/>
+<wire x1="156.21" y1="231.14" x2="156.21" y2="228.6" width="0.1524" layer="91"/>
+<junction x="156.21" y="228.6"/>
+<pinref part="C29" gate="G$1" pin="2"/>
+<wire x1="161.29" y1="229.87" x2="161.29" y2="228.6" width="0.1524" layer="91"/>
+<junction x="161.29" y="228.6"/>
+</segment>
+</net>

Commit message: switched to smaller jst connector and done routing
Parts:
- added U$7: JST-ZR-2, Mine:JST-ZR-2
- added U$8: JST-ZR-2SMD, Mine:JST-ZR-2SMD
- added X4: S4B-ZR, con-jst:S4B-ZR
Connections:
- net GND: now also S4.1, U$7.2, U$8.2
- net N$2: now also U$7.1, U$8.1
Other:
- moved on the sheet: JP1
Changed lines of the file:
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@@
 <part name="GND54" library="SparkFun" deviceset="GND" device=""/>
 <part name="RN1" library="resistor-dil" deviceset="4R-N" device="0402ARV341"/>
+<part name="X4" library="con-jst" deviceset="?4B-ZR" device="S"/>
+<part name="U$7" library="Mine" deviceset="JST-ZR-2" device=""/>
+<part name="U$8" library="Mine" deviceset="JST-ZR-2" device="SMD"/>
+<part name="GND55" library="SparkFun" deviceset="GND" device=""/>
+<part name="GND56" library="SparkFun" deviceset="GND" device=""/>
+<part name="GND57" library="supply1" deviceset="GND" device=""/>
 </parts>
 <sheets>
 <sheet>
 <plain>
-<text x="144.78" y="248.92" size="1.778" layer="91">CHECK!!!</text>
+<text x="132.08" y="248.92" size="1.778" layer="91">CHECK!!!</text>
 <text x="200.66" y="229.87" size="1.778" layer="91">connect -&gt; ?</text>
 <text x="209.55" y="41.91" size="1.778" layer="91">connect -&gt; ?</text>
@@
 <instance part="U$3" gate="G$1" x="241.3" y="52.07"/>
 <instance part="U$4" gate="G$1" x="240.03" y="161.29"/>
-<instance part="JP1" gate="G$1" x="147.32" y="243.84" rot="R270"/>
+<instance part="JP1" gate="G$1" x="147.32" y="248.92" rot="R270"/>
 <instance part="IC1" gate="G$1" x="53.34" y="160.02"/>
 <instance part="X1" gate="G$1" x="-29.21" y="170.18" rot="MR0"/>
@@
 <instance part="RN1" gate="C" x="281.94" y="66.04"/>
 <instance part="RN1" gate="D" x="281.94" y="60.96"/>
+<instance part="X4" gate="-1" x="147.32" y="264.16" rot="R90"/>
+<instance part="X4" gate="-2" x="149.86" y="264.16" rot="R90"/>
+<instance part="X4" gate="-3" x="152.4" y="264.16" rot="R90"/>
+<instance part="X4" gate="-4" x="154.94" y="264.16" rot="R90"/>
+<instance part="U$7" gate="G$1" x="165.1" y="254" rot="R270"/>
+<instance part="U$8" gate="G$1" x="177.8" y="254" rot="R270"/>
+<instance part="GND55" gate="1" x="167.64" y="243.84" smashed="yes"/>
+<instance part="GND56" gate="1" x="180.34" y="243.84" smashed="yes"/>
+<instance part="GND57" gate="1" x="96.52" y="171.45" rot="R90"/>
 </instances>
 <busses>
@@
 <pinref part="JP1" gate="G$1" pin="1"/>
 <pinref part="GND15" gate="1" pin="GND"/>
+<wire x1="147.32" y1="241.3" x2="147.32" y2="236.22" width="0.1524" layer="91"/>
 </segment>
 <segment>
@@
 <pinref part="C29" gate="G$1" pin="1"/>
 <pinref part="GND54" gate="1" pin="GND"/>
+</segment>
+<segment>
+<pinref part="U$7" gate="G$1" pin="2"/>
+<pinref part="GND55" gate="1" pin="GND"/>
+</segment>
+<segment>
+<pinref part="U$8" gate="G$1" pin="2"/>
+<pinref part="GND56" gate="1" pin="GND"/>
+</segment>
+<segment>
+<pinref part="S4" gate="G$1" pin="1"/>
+<pinref part="GND57" gate="1" pin="GND"/>
 </segment>
 </net>
@@
 <pinref part="JP1" gate="G$1" pin="2"/>
 <wire x1="139.7" y1="228.6" x2="149.86" y2="228.6" width="0.1524" layer="91"/>
-<wire x1="149.86" y1="236.22" x2="149.86" y2="228.6" width="0.1524" layer="91"/>
+<wire x1="149.86" y1="241.3" x2="149.86" y2="228.6" width="0.1524" layer="91"/>
 <pinref part="S1" gate="G$1" pin="1"/>
 <wire x1="139.7" y1="209.55" x2="139.7" y2="214.63" width="0.1524" layer="91"/>
@@
 <pinref part="D2" gate="G$1" pin="A"/>
 <junction x="149.86" y="228.6"/>
+<pinref part="U$7" gate="G$1" pin="1"/>
+<wire x1="149.86" y1="241.3" x2="165.1" y2="241.3" width="0.1524" layer="91"/>
+<wire x1="165.1" y1="241.3" x2="165.1" y2="246.38" width="0.1524" layer="91"/>
+<pinref part="U$8" gate="G$1" pin="1"/>
+<wire x1="165.1" y1="241.3" x2="177.8" y2="241.3" width="0.1524" layer="91"/>
+<wire x1="177.8" y1="241.3" x2="177.8" y2="246.38" width="0.1524" layer="91"/>
 </segment>
 </net>

Commit message: some routing done, changed lipo charger
Parts:
- removed U1: MAX1555, SparkFun:MAX1555
- added C30: (no value), resistor:C-EUC0402
- added R14: (no value), rcl:R-EU_R0402
- added U2: MCP73831, SparkFun-PowerIC:MCP73831
Connections:
- new net N$33: R14.1, U2.PROG
- net +3V3: now also C30.1, U$1.CS, U$1.SA0_SDO
- net GND: now also C30.2, R14.2, U2.VSS; no longer U$1.SA0_SDO, U1.GND
- net N$1: now also U2.VIN; no longer U1.USB
- net N$10: now also U2.STAT; no longer U1.CHG
- net N$2: now also U2.VBAT; no longer U1.BATT
Changed lines of the file:
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@@
 <layer number="106" name="bPlate" color="7" fill="1" visible="yes" active="yes"/>
 <layer number="107" name="Crop" color="7" fill="1" visible="yes" active="yes"/>
+<layer number="108" name="tplace-old" color="10" fill="1" visible="yes" active="yes"/>
+<layer number="109" name="ref-old" color="11" fill="1" visible="yes" active="yes"/>
 <layer number="116" name="Patch_BOT" color="9" fill="4" visible="yes" active="yes"/>
 <layer number="121" name="_tsilk" color="7" fill="1" visible="yes" active="yes"/>
@@
 <layer number="144" name="Drill_legend" color="7" fill="1" visible="yes" active="yes"/>
 <layer number="151" name="HeatSink" color="7" fill="1" visible="yes" active="yes"/>
+<layer number="199" name="Contour" color="7" fill="1" visible="yes" active="yes"/>
 <layer number="200" name="200bmp" color="1" fill="10" visible="yes" active="yes"/>
 <layer number="201" name="201bmp" color="2" fill="10" visible="yes" active="yes"/>
@@
 <part name="IC1" library="Mine" deviceset="CC430F513X" device=""/>
 <part name="X1" library="Mine" deviceset="0896BM15A0001" device=""/>
-<part name="U1" library="SparkFun" deviceset="MAX1555" device=""/>
 <part name="LED1" library="SparkFun" deviceset="LED" device="0603"/>
 <part name="LED2" library="SparkFun" deviceset="LED" device="0603"/>
@@
 <part name="X2" library="SparkFun" deviceset="USB" device="-MICROB"/>
 <part name="GND32" library="SparkFun" deviceset="GND" device=""/>
-<part name="GND13" library="SparkFun" deviceset="GND" device=""/>
 <part name="C11" library="resistor" deviceset="C-EU" device="C0402"/>
 <part name="GND14" library="SparkFun" deviceset="GND" device=""/>
@@
 <part name="C27" library="resistor" deviceset="C-EU" device="C0402"/>
 <part name="GND49" library="SparkFun" deviceset="GND" device=""/>
-<part name="GND50" library="SparkFun" deviceset="GND" device=""/>
 <part name="GND51" library="SparkFun" deviceset="GND" device=""/>
 <part name="C28" library="resistor" deviceset="C-EU" device="C0402"/>
@@
 <part name="GND56" library="SparkFun" deviceset="GND" device=""/>
 <part name="GND57" library="supply1" deviceset="GND" device=""/>
+<part name="U2" library="SparkFun-PowerIC" deviceset="MCP73831" device=""/>
+<part name="R14" library="rcl" deviceset="R-EU_" device="R0402"/>
+<part name="GND13" library="SparkFun" deviceset="GND" device=""/>
+<part name="GND58" library="SparkFun" deviceset="GND" device=""/>
+<part name="C30" library="resistor" deviceset="C-EU" device="C0402"/>
+<part name="GND59" library="SparkFun" deviceset="GND" device=""/>
+<part name="+3V17" library="supply1" deviceset="+3V3" device=""/>
+<part name="+3V18" library="supply1" deviceset="+3V3" device=""/>
 </parts>
 <sheets>
@@
 <instance part="IC1" gate="G$1" x="53.34" y="160.02"/>
 <instance part="X1" gate="G$1" x="-29.21" y="170.18" rot="MR0"/>
-<instance part="U1" gate="G$1" x="124.46" y="226.06"/>
 <instance part="LED1" gate="G$1" x="100.33" y="149.86" rot="R90"/>
 <instance part="LED2" gate="G$1" x="100.33" y="146.05" rot="R90"/>
@@
 <instance part="X2" gate="G$1" x="96.52" y="229.87" rot="R180"/>
 <instance part="GND32" gate="1" x="100.33" y="238.76" smashed="yes" rot="R180"/>
-<instance part="GND13" gate="1" x="106.68" y="226.06" smashed="yes" rot="R270"/>
 <instance part="C11" gate="G$1" x="105.41" y="233.68" rot="MR0"/>
 <instance part="GND14" gate="1" x="105.41" y="238.76" smashed="yes" rot="R180"/>
@@
 <instance part="C27" gate="G$1" x="132.08" y="191.77" rot="MR0"/>
 <instance part="GND49" gate="1" x="132.08" y="184.15" smashed="yes"/>
-<instance part="GND50" gate="1" x="218.44" y="218.44" smashed="yes" rot="R270"/>
 <instance part="GND51" gate="1" x="218.44" y="49.53" smashed="yes" rot="R270"/>
 <instance part="C28" gate="G$1" x="-10.16" y="110.49" rot="MR180"/>
@@
 <instance part="GND56" gate="1" x="180.34" y="243.84" smashed="yes"/>
 <instance part="GND57" gate="1" x="96.52" y="171.45" rot="R90"/>
+<instance part="U2" gate="G$1" x="121.92" y="226.06"/>
+<instance part="R14" gate="G$1" x="137.16" y="215.9" rot="R270"/>
+<instance part="GND13" gate="1" x="134.62" y="223.52" smashed="yes" rot="R90"/>
+<instance part="GND58" gate="1" x="137.16" y="208.28" smashed="yes"/>
+<instance part="C30" gate="G$1" x="191.77" y="133.35" rot="MR180"/>
+<instance part="GND59" gate="1" x="191.77" y="140.97" smashed="yes" rot="R180"/>
+<instance part="+3V17" gate="G$1" x="220.98" y="226.06" rot="R90"/>
+<instance part="+3V18" gate="G$1" x="220.98" y="218.44" rot="R90"/>
 </instances>
 <busses>
@@
 </segment>
 <segment>
-<pinref part="U1" gate="G$1" pin="GND"/>
-<pinref part="GND13" gate="1" pin="GND"/>
-</segment>
-<segment>
 <pinref part="C11" gate="G$1" pin="1"/>
 <pinref part="GND14" gate="1" pin="GND"/>
@@
 </segment>
 <segment>
-<pinref part="U$1" gate="G$1" pin="SA0_SDO"/>
-<wire x1="223.52" y1="218.44" x2="220.98" y2="218.44" width="0.1524" layer="91"/>
-<pinref part="GND50" gate="1" pin="GND"/>
-</segment>
-<segment>
 <pinref part="U$3" gate="G$1" pin="SA0"/>
 <wire x1="223.52" y1="49.53" x2="220.98" y2="49.53" width="0.1524" layer="91"/>
@@
 <pinref part="S4" gate="G$1" pin="1"/>
 <pinref part="GND57" gate="1" pin="GND"/>
+</segment>
+<segment>
+<pinref part="U2" gate="G$1" pin="VSS"/>
+<pinref part="GND13" gate="1" pin="GND"/>
+</segment>
+<segment>
+<pinref part="R14" gate="G$1" pin="2"/>
+<pinref part="GND58" gate="1" pin="GND"/>
+</segment>
+<segment>
+<pinref part="C30" gate="G$1" pin="2"/>
+<pinref part="GND59" gate="1" pin="GND"/>
 </segment>
 </net>
@@
 <wire x1="102.87" y1="227.33" x2="105.41" y2="227.33" width="0.1524" layer="91"/>
 <wire x1="105.41" y1="227.33" x2="105.41" y2="228.6" width="0.1524" layer="91"/>
-<pinref part="U1" gate="G$1" pin="USB"/>
 <wire x1="105.41" y1="228.6" x2="109.22" y2="228.6" width="0.1524" layer="91"/>
 <pinref part="C11" gate="G$1" pin="2"/>
@@
 <wire x1="156.21" y1="254" x2="109.22" y2="254" width="0.1524" layer="91"/>
 <wire x1="109.22" y1="254" x2="109.22" y2="228.6" width="0.1524" layer="91"/>
+<pinref part="U2" gate="G$1" pin="VIN"/>
+<wire x1="111.76" y1="228.6" x2="109.22" y2="228.6" width="0.1524" layer="91"/>
 <junction x="109.22" y="228.6"/>
 </segment>
@@
 <net name="N$2" class="0">
 <segment>
-<pinref part="U1" gate="G$1" pin="BATT"/>
-<wire x1="137.16" y1="228.6" x2="139.7" y2="228.6" width="0.1524" layer="91"/>
 <pinref part="JP1" gate="G$1" pin="2"/>
 <wire x1="139.7" y1="228.6" x2="149.86" y2="228.6" width="0.1524" layer="91"/>
@@
 <wire x1="165.1" y1="241.3" x2="177.8" y2="241.3" width="0.1524" layer="91"/>
 <wire x1="177.8" y1="241.3" x2="177.8" y2="246.38" width="0.1524" layer="91"/>
+<pinref part="U2" gate="G$1" pin="VBAT"/>
+<wire x1="132.08" y1="228.6" x2="139.7" y2="228.6" width="0.1524" layer="91"/>
+<junction x="149.86" y="241.3"/>
+<junction x="165.1" y="241.3"/>
 </segment>
 </net>
@@
 <pinref part="U$6" gate="G$1" pin="VCC"/>
 <pinref part="+3V12" gate="G$1" pin="+3V3"/>
+<pinref part="C30" gate="G$1" pin="1"/>
+<junction x="191.77" y="130.81"/>
+<pinref part="C30" gate="G$1" pin="1"/>
 </segment>
 <segment>
@@
 <pinref part="+3V16" gate="G$1" pin="+3V3"/>
 <pinref part="JP3" gate="G$1" pin="1"/>
+</segment>
+<segment>
+<pinref part="U$1" gate="G$1" pin="CS"/>
+<pinref part="+3V17" gate="G$1" pin="+3V3"/>
+</segment>
+<segment>
+<pinref part="U$1" gate="G$1" pin="SA0_SDO"/>
+<pinref part="+3V18" gate="G$1" pin="+3V3"/>
 </segment>
 </net>
@@
 </segment>
 </net>
-<net name="N$10" class="0">
-<segment>
-<pinref part="U1" gate="G$1" pin="CHG"/>
-<pinref part="R13" gate="G$1" pin="1"/>
-</segment>
-</net>
 <net name="N$18" class="0">
 <segment>
@@
 </segment>
 </net>
+<net name="N$10" class="0">
+<segment>
+<pinref part="U2" gate="G$1" pin="STAT"/>
+<pinref part="R13" gate="G$1" pin="1"/>
+<wire x1="111.76" y1="223.52" x2="109.22" y2="223.52" width="0.1524" layer="91"/>
+</segment>
+</net>
+<net name="N$33" class="0">
+<segment>
+<pinref part="U2" gate="G$1" pin="PROG"/>
+<pinref part="R14" gate="G$1" pin="1"/>
+<wire x1="132.08" y1="226.06" x2="137.16" y2="226.06" width="0.1524" layer="91"/>
+<wire x1="137.16" y1="226.06" x2="137.16" y2="220.98" width="0.1524" layer="91"/>
+</segment>
+</net>

Commit message: finishing off, almost done
Parts:
- removed JP1: (no value), SparkFun:M02-JST-2MM-SMT
- removed RN1: (no value), resistor-dil:4R-N0402ARV341
- removed U$5: SPI_FLASH-X25XXSMD, SparkFun:SPI_FLASH-X25XXSMD
- removed X4: S4B-ZR, con-jst:S4B-ZR
Connections:
- removed net N$27: U$6.WP
- net +3V3: now also U$6.WP
- net GND: no longer JP1.1
- net N$2: no longer JP1.2
Other:
- moved on the sheet: JP2, L1, LED1, LED2, LED3, LED4, R11, R12, R2, R3, S4
