File: rocket-logger.brd (EAGLE design)
At the start: 58.5 x 62 mm, 80 parts, among them IC1 CC430F513X, U2 MCP73831, X1 0896BM15A0001, X2 USB-MICROB, X3 SMA-142-0701-801/806, X4 S4B-ZR

Commit message: fixing some drc
Parts:
- moved C13 0.05 mm to (2.61, 8.56)
- moved C3 0.05 mm to (2.61, 9.70)
Routing:
- net +3V3: track 125.6 -> 124.0 mm

Commit message: finishing off, almost done
Parts:
- removed JP1: (no value), SparkFun:S2B-PH
- removed RN1: (no value), resistor-dil:4X0402ARV341
- removed U$5: SPI_FLASH-X25XXSMD, SparkFun:SO08
- removed X4: S4B-ZR, con-jst:S4B-ZR
- moved R5 0.11 mm to (15.9, 27.1)
- turned S4 to 0 degrees
Connections:
- removed net N$27: U$6.3
- net +3V3: now also U$6.3
- net GND: no longer JP1.1
- net N$2: no longer JP1.2
Routing:
- net N$28: track 37.7 -> 28.2 mm
- net GND: track 145.1 -> 140.1 mm, vias 45 -> 59
- net +3V3: track 124.0 -> 125.2 mm
- net AVCC_RF2: track 20.2 -> 19.5 mm
- net N$12: track 10.8 -> 11.5 mm, vias 0 -> 1
- net N$24: track 40.9 -> 40.4 mm
Other:
- board text added: "V1 JAN 14"
- board text removed: "1"
- board text removed: "2"
- board text removed: "SUSF"
- board text removed: "V1 NOV 13"
- board text removed: "untent and label"

Commit message: minor change
Parts:
- moved C18 0.15 mm to (7.92, 30.3)
Routing:
- net GND: track 140.1 -> 139.5 mm
Changed lines of the file:
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@@
 <layer number="19" name="Unrouted" color="6" fill="1" visible="yes" active="yes"/>
 <layer number="20" name="Dimension" color="15" fill="1" visible="yes" active="yes"/>
-<layer number="21" name="tPlace" color="16" fill="1" visible="no" active="yes"/>
+<layer number="21" name="tPlace" color="16" fill="1" visible="yes" active="yes"/>
 <layer number="22" name="bPlace" color="14" fill="1" visible="yes" active="yes"/>
 <layer number="23" name="tOrigins" color="15" fill="1" visible="yes" active="yes"/>
@@
 <param name="mdViaViaSameLayer" value="8mil"/>
 <param name="mnLayersViaInSmd" value="2"/>
-<param name="mdCopperDimension" value="10mil"/>
+<param name="mdCopperDimension" value="0mil"/>
 <param name="mdDrill" value="10mil"/>
 <param name="mdSmdStop" value="0mil"/>
@@
 <element name="C16" library="resistor" package="C0402" value="100n" x="0.8128" y="10.25" rot="R90"/>
 <element name="C17" library="resistor" package="C0402" value="" x="2" y="18" rot="R180"/>
-<element name="C18" library="resistor" package="C0402" value="1u" x="7.92" y="30.1752" rot="R180"/>
+<element name="C18" library="resistor" package="C0402" value="1u" x="7.92" y="30.3276" rot="R180"/>
 <element name="C19" library="resistor" package="C0402" value="1u" x="4.75" y="30.2032" rot="R180"/>
 <element name="C20" library="resistor" package="C0402" value="100n" x="2.064" y="19.358" rot="R180"/>
@@
 <via x="13.8176" y="27.6352" extent="1-16" drill="0.381" shape="octagon"/>
 <polygon width="0.2032" layer="16" isolate="0.254">
-<vertex x="1.6256" y="49.9872"/>
-<vertex x="16.8656" y="49.9872"/>
-<vertex x="16.8656" y="0"/>
-<vertex x="0" y="0"/>
-<vertex x="0" y="48.768"/>
-<vertex x="1.2192" y="49.9872"/>
+<vertex x="2.032" y="49.5808"/>
+<vertex x="16.6624" y="49.5808"/>
+<vertex x="16.6624" y="0.4064"/>
+<vertex x="0.4064" y="0.4064"/>
+<vertex x="0.4064" y="35.56"/>
+<vertex x="1.8288" y="36.3728"/>
+<vertex x="1.8288" y="45.1104"/>
+<vertex x="0.6096" y="45.3136"/>
+<vertex x="0.6096" y="48.768"/>
 </polygon>
 <wire x1="2.714" y1="18.064" x2="2.65" y2="18" width="0.2032" layer="1"/>
@@
 <via x="9.9568" y="31.2928" extent="1-16" drill="0.381" shape="octagon"/>
 <wire x1="9.9568" y1="31.2928" x2="10.16" y2="31.2928" width="0.2032" layer="16"/>
-<via x="7.7724" y="32.1056" extent="1-16" drill="0.381" shape="octagon"/>
-<wire x1="7.7724" y1="32.1056" x2="7.112" y2="32.1056" width="0.2032" layer="16"/>
+<via x="7.7724" y="32.1564" extent="1-16" drill="0.381" shape="octagon"/>
 <via x="9.2964" y="36.1696" extent="1-16" drill="0.381" shape="octagon"/>
 <via x="4.8768" y="32.2072" extent="1-16" drill="0.381" shape="octagon"/>
@@
 <wire x1="5.4" y1="30.2032" x2="5.236" y2="30.2032" width="0.2032" layer="1"/>
 <wire x1="5.236" y1="30.2032" x2="5.2164" y2="30.1836" width="0.2032" layer="1"/>
-<wire x1="7.7724" y1="32.1056" x2="7.7724" y2="32.3942" width="0.2032" layer="1"/>
+<wire x1="7.7724" y1="32.1564" x2="7.7724" y2="32.3942" width="0.2032" layer="1"/>
 <wire x1="7.7724" y1="32.3942" x2="8.0542" y2="32.676" width="0.2032" layer="1"/>
 <wire x1="11.0542" y1="33.176" x2="11.84" y2="33.176" width="0.2032" layer="1"/>
@@
 <wire x1="11.0542" y1="34.176" x2="11.9504" y2="34.176" width="0.2032" layer="1"/>
 <wire x1="11.9504" y1="34.176" x2="11.9888" y2="34.1376" width="0.2032" layer="1"/>
-<wire x1="8.5344" y1="30.1396" x2="8.57" y2="30.1752" width="0.2032" layer="1"/>
 <wire x1="1.9556" y1="10.8008" x2="2.0064" y2="10.8516" width="0.2032" layer="1"/>
 <wire x1="9.5542" y1="31.8986" x2="9.5542" y2="31.6954" width="0.254" layer="1"/>
@@
 <wire x1="10.9728" y1="18.6944" x2="10.988640625" y2="18.6944" width="0.4064" layer="1"/>
 <wire x1="10.988640625" y1="18.6944" x2="11.337290625" y2="19.04305" width="0.4064" layer="1"/>
+<wire x1="8.5344" y1="30.1396" x2="8.5344" y2="30.292" width="0.2032" layer="1"/>
+<wire x1="8.5344" y1="30.292" x2="8.57" y2="30.3276" width="0.2032" layer="1"/>
 <wire x1="15.0368" y1="14.8336" x2="18.064" y2="13.1492" width="0" layer="19" extent="1-16"/>
+<wire x1="16.0528" y1="3.048" x2="14.9196" y2="2.5654" width="0" layer="19" extent="1-1"/>
+<wire x1="16.3576" y1="1.6764" x2="16.0528" y2="3.048" width="0" layer="19" extent="1-1"/>
 </signal>
 <signal name="VCORE">
@@
 <wire x1="14.478" y1="26.2828" x2="14.6632" y2="26.468" width="0.2032" layer="1"/>
 <polygon width="0.2032" layer="1">
-<vertex x="15.8496" y="39.8272"/>
+<vertex x="16.4592" y="39.8272"/>
 <vertex x="10.7696" y="39.8272"/>
 <vertex x="10.5664" y="37.1856"/>
-<vertex x="0.2032" y="37.1856"/>
+<vertex x="1.8288" y="36.1696"/>
+<vertex x="1.4224" y="36.1696"/>
+<vertex x="0.4064" y="35.3568"/>
 <vertex x="0.6096" y="10.3632"/>
-<vertex x="17.0688" y="10.5664"/>
-<vertex x="15.8496" y="33.9344"/>
+<vertex x="16.6624" y="10.5664"/>
+<vertex x="16.6624" y="39.4208"/>
 </polygon>
 <wire x1="10.7696" y1="29.266" x2="10.7696" y2="29.8704" width="0.4064" layer="1"/>
@@
 <wire x1="16.4592" y1="10.5664" x2="16.4592" y2="8.8504" width="0.4064" layer="1"/>
 <wire x1="16.4592" y1="8.8504" x2="15.94" y2="8.3312" width="0.4064" layer="1"/>
+<wire x1="5.6896" y1="35.7632" x2="4.9856" y2="36.096" width="0" layer="19" extent="1-16"/>
 </signal>
 <signal name="N$3">
@@
 <wire x1="7.3152" y1="29.2608" x2="7.3152" y2="30.0736" width="0.4064" layer="1"/>
 <wire x1="7.3152" y1="30.0736" x2="7.3152" y2="30.13" width="0.4064" layer="1"/>
-<wire x1="7.27" y1="30.1752" x2="7.1684" y2="30.0736" width="0.2032" layer="1"/>
 <wire x1="7.1684" y1="30.0736" x2="7.3152" y2="30.0736" width="0.2032" layer="1"/>
+<wire x1="7.1684" y1="30.0736" x2="7.1684" y2="30.226" width="0.2032" layer="1"/>
+<wire x1="7.1684" y1="30.226" x2="7.27" y2="30.3276" width="0.2032" layer="1"/>
 </signal>
 <signal name="N$15">
@@
 <wire x1="4.4196" y1="14.6812" x2="2.794" y2="14.6812" width="0.2032" layer="16"/>
 <wire x1="2.794" y1="14.6812" x2="1.2192" y2="16.256" width="0.2032" layer="16"/>
-<wire x1="9.3472" y1="30.6832" x2="9.3472" y2="29.1852" width="0.2032" layer="1"/>
+<wire x1="9.3472" y1="30.8864" x2="9.3472" y2="29.1852" width="0.2032" layer="1"/>
 <wire x1="3.26" y1="15.285" x2="3.8158" y2="15.285" width="0.2032" layer="1"/>
 <wire x1="3.8158" y1="15.285" x2="4.4196" y2="14.6812" width="0.2032" layer="1"/>
@@
 <wire x1="2.5908" y1="29.8704" x2="2.6416" y2="29.9212" width="0.2032" layer="16"/>
 <wire x1="2.6416" y1="29.9212" x2="5.5372" y2="29.9212" width="0.2032" layer="16"/>
-<via x="7.9248" y="31.0896" extent="1-16" drill="0.381" shape="octagon"/>
-<wire x1="7.9248" y1="31.0896" x2="8.5344" y2="31.0896" width="0.2032" layer="1"/>
-<wire x1="8.5344" y1="31.0896" x2="8.7376" y2="31.2928" width="0.2032" layer="1"/>
-<wire x1="8.7376" y1="31.2928" x2="9.0542" y2="31.6094" width="0.2032" layer="1"/>
-<wire x1="9.0542" y1="32.176" x2="9.0542" y2="31.6094" width="0.2032" layer="1"/>
-<wire x1="9.3472" y1="30.6832" x2="8.7376" y2="31.2928" width="0.2032" layer="1"/>
-<wire x1="7.9248" y1="31.0896" x2="6.7056" y2="31.0896" width="0.2032" layer="16"/>
-<wire x1="6.7056" y1="31.0896" x2="5.5372" y2="29.9212" width="0.2032" layer="16"/>
+<via x="7.9248" y="31.242" extent="1-16" drill="0.381" shape="octagon"/>
+<wire x1="9.0542" y1="32.176" x2="9.0542" y2="31.3046" width="0.2032" layer="1"/>
+<wire x1="6.858" y1="31.242" x2="5.5372" y2="29.9212" width="0.2032" layer="16"/>
 <wire x1="9.3472" y1="29.1852" x2="9.4092" y2="29.1232" width="0.2032" layer="1"/>
 <wire x1="2.1168" y1="31.29" x2="2.1168" y2="31.0048" width="0.2032" layer="1"/>
 <wire x1="2.1168" y1="31.0048" x2="2.1336" y2="30.988" width="0.2032" layer="1"/>
 <wire x1="2.1336" y1="30.988" x2="2.1336" y2="30.4292" width="0.2032" layer="1"/>
+<wire x1="9.3472" y1="30.8864" x2="8.9916" y2="31.242" width="0.2032" layer="1"/>
+<wire x1="7.9248" y1="31.242" x2="8.9916" y2="31.242" width="0.2032" layer="1"/>
+<wire x1="9.0542" y1="31.3046" x2="8.9916" y2="31.242" width="0.2032" layer="1"/>
+<wire x1="7.9248" y1="31.242" x2="6.858" y2="31.242" width="0.2032" layer="16"/>
 </signal>
 <signal name="SCL">
@@
 <wire x1="1.9304" y1="29.21" x2="0.4572" y2="29.21" width="0.2032" layer="1"/>
 <wire x1="0.4572" y1="29.21" x2="0.4064" y2="29.2608" width="0.2032" layer="1"/>
-<wire x1="6.35" y1="29.8196" x2="6.35" y2="30.5308" width="0.2032" layer="1"/>
-<wire x1="6.35" y1="30.5308" x2="7.112" y2="31.2928" width="0.2032" layer="1"/>
+<wire x1="6.35" y1="29.8196" x2="6.35" y2="30.734" width="0.2032" layer="1"/>
 <wire x1="7.112" y1="31.2928" x2="7.112" y2="32.9184" width="0.2032" layer="1"/>
 <wire x1="8.0542" y1="33.176" x2="7.3696" y2="33.176" width="0.2032" layer="1"/>
@@
 <wire x1="5.7404" y1="29.21" x2="6.35" y2="29.8196" width="0.2032" layer="16"/>
 <wire x1="1.9304" y1="29.21" x2="5.7404" y2="29.21" width="0.2032" layer="16"/>
+<wire x1="6.35" y1="30.734" x2="6.7056" y2="31.0896" width="0.2032" layer="1"/>
+<wire x1="6.7056" y1="31.0896" x2="6.9088" y2="31.0896" width="0.2032" layer="1"/>
+<wire x1="6.9088" y1="31.0896" x2="7.112" y2="31.2928" width="0.2032" layer="1"/>
 </signal>
 <signal name="KEEPON">
