File: rocket-logger-merged.brd (EAGLE design)
At the start: 50 x 50 mm, 127 parts, among them IC1 CC430F513X, IC3 CC430F513X, U2 MCP73831, U3 MCP73831, X1 0896BM15A0001, X2 USB-MICROB, X3 SMA-142-0701-801/806, X4 0896BM15A0001, X5 USB-MICROB, X6 SMA-142-0701-801/806

Commit message: sent off
Routing:
- net GND1: track 139.5 -> 142.9 mm
- net GND: track 74.5 -> 71.4 mm
- net N$3: track 2.36 -> 0.95 mm
- net +3V3: track 63.9 -> 64.8 mm
- net AVCC_RF2: track 18.3 -> 19.1 mm
- net +3V1: track 125.2 -> 125.8 mm
