File: rocket-logger-basic.sch (EAGLE design)
At the start: 51 parts, among them IC1 CC430F513X, U1 MAX1555, X1 0896BM15A0001, X2 USB-MICROB, X3 SMA-142-0701-801/806

Commit message: added charging led
Parts:
- removed S4: SWITCH-MOMENTARY-2SMD, SparkFun:SWITCH-MOMENTARY-2SMD
- removed SV1: (no value), con-lstb:MA04-1
- added JP3: (no value), SparkFun:M04PTH
- added LED3: (no value), SparkFun:LED0603
- added R11: (no value), rcl:R-EU_R0402
Connections:
- new net INT2: IC1.P3.4, U$4.INT1
- new net N$15: R11.1, U1.CHG
- new net N$18: LED3.C, R11.2
- net +3V3: now also JP3.1
- net GND: now also JP3.2
- net N$1: now also LED3.A
- net N$23: now also JP3.4; no longer SV1.4
- net N$26: now also JP3.3; no longer SV1.3
Other:
- note added: "3"
- note added: "what happens when charging?"
Changed lines of the file:
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@@
 <part name="X3" library="con-coax" deviceset="SMA-" device="142-0701-801/806"/>
 <part name="GND22" library="supply1" deviceset="GND" device=""/>
-<part name="SV1" library="con-lstb" deviceset="MA04-1" device=""/>
 <part name="R2" library="rcl" deviceset="R-EU_" device="R0402"/>
 <part name="R3" library="rcl" deviceset="R-EU_" device="R0402"/>
@@
 <part name="R5" library="rcl" deviceset="R-EU_" device="R0402"/>
 <part name="SG1" library="buzzer" deviceset="EFB?" device="RD24C411"/>
-<part name="S4" library="SparkFun" deviceset="SWITCH-MOMENTARY-2" device="SMD"/>
 <part name="C26" library="resistor" deviceset="C-EU" device="C0402"/>
 <part name="GND46" library="SparkFun" deviceset="GND" device=""/>
@@
 <part name="GND29" library="supply1" deviceset="GND" device=""/>
 <part name="+3V2" library="supply1" deviceset="+3V3" device=""/>
+<part name="GND30" library="supply1" deviceset="GND" device=""/>
+<part name="+3V3" library="supply1" deviceset="+3V3" device=""/>
+<part name="JP3" library="SparkFun" deviceset="M04" device="PTH"/>
+<part name="R11" library="rcl" deviceset="R-EU_" device="R0402"/>
+<part name="LED3" library="SparkFun" deviceset="LED" device="0603"/>
 </parts>
 <sheets>
@@
 <text x="144.78" y="248.92" size="1.778" layer="91">CHECK!!!</text>
 <text x="209.55" y="153.67" size="1.778" layer="91">connect -&gt; ?</text>
+<text x="232.664" y="144.018" size="1.778" layer="91">3</text>
+<text x="109.22" y="245.11" size="1.778" layer="91">what happens when charging?</text>
 </plain>
 <instances>
@@
 <instance part="X3" gate="G1" x="-49.53" y="172.72"/>
 <instance part="GND22" gate="1" x="-46.99" y="167.64"/>
-<instance part="SV1" gate="1" x="-22.86" y="115.57"/>
 <instance part="R2" gate="G$1" x="92.71" y="149.86"/>
 <instance part="R3" gate="G$1" x="92.71" y="146.05"/>
@@
 <instance part="R5" gate="G$1" x="168.91" y="191.77" rot="R180"/>
 <instance part="SG1" gate="G$1" x="101.6" y="134.62" rot="R270"/>
-<instance part="S4" gate="G$1" x="88.9" y="171.45" rot="R180"/>
 <instance part="C26" gate="G$1" x="139.7" y="233.68" rot="MR0"/>
 <instance part="GND46" gate="1" x="139.7" y="238.76" smashed="yes" rot="R180"/>
@@
 <instance part="GND29" gate="1" x="-11.43" y="102.87"/>
 <instance part="+3V2" gate="G$1" x="-11.43" y="133.35"/>
+<instance part="GND30" gate="1" x="-12.7" y="113.03" rot="R90"/>
+<instance part="+3V3" gate="G$1" x="-12.7" y="110.49" rot="R270"/>
+<instance part="JP3" gate="G$1" x="-20.32" y="113.03"/>
+<instance part="R11" gate="G$1" x="109.22" y="212.09" rot="R270"/>
+<instance part="LED3" gate="G$1" x="109.22" y="201.93" rot="R180"/>
 </instances>
 <busses>
@@
 <pinref part="GND29" gate="1" pin="GND"/>
 </segment>
+<segment>
+<pinref part="GND30" gate="1" pin="GND"/>
+<pinref part="JP3" gate="G$1" pin="2"/>
+</segment>
 </net>
 <net name="N$1" class="0">
 <segment>
 <pinref part="X2" gate="G$1" pin="VBUS"/>
-<wire x1="99.06" y1="227.33" x2="105.41" y2="227.33" width="0.1524" layer="91"/>
+<wire x1="99.06" y1="227.33" x2="101.6" y2="227.33" width="0.1524" layer="91"/>
+<wire x1="101.6" y1="227.33" x2="105.41" y2="227.33" width="0.1524" layer="91"/>
 <wire x1="105.41" y1="227.33" x2="105.41" y2="228.6" width="0.1524" layer="91"/>
 <pinref part="U1" gate="G$1" pin="USB"/>
@@
 <pinref part="C11" gate="G$1" pin="2"/>
 <junction x="105.41" y="228.6"/>
+<pinref part="LED3" gate="G$1" pin="A"/>
+<wire x1="109.22" y1="199.39" x2="101.6" y2="199.39" width="0.1524" layer="91"/>
+<wire x1="101.6" y1="199.39" x2="101.6" y2="227.33" width="0.1524" layer="91"/>
+<junction x="101.6" y="227.33"/>
 </segment>
 </net>
@@
 <pinref part="+3V2" gate="G$1" pin="+3V3"/>
 </segment>
+<segment>
+<pinref part="+3V3" gate="G$1" pin="+3V3"/>
+<pinref part="JP3" gate="G$1" pin="1"/>
+</segment>
 </net>
 <net name="N$3" class="0">
@@
 <wire x1="-2.54" y1="162.56" x2="-3.81" y2="163.83" width="0.1524" layer="91"/>
 <wire x1="-3.81" y1="163.83" x2="-6.35" y2="163.83" width="0.1524" layer="91"/>
+<junction x="-6.35" y="163.83"/>
 </segment>
 </net>
@@
 <wire x1="-3.81" y1="158.75" x2="-2.54" y2="160.02" width="0.1524" layer="91"/>
 <pinref part="IC1" gate="G$1" pin="RF_XOUT"/>
+<junction x="-6.35" y="158.75"/>
 </segment>
 </net>
@@
 <segment>
 <pinref part="IC1" gate="G$1" pin="TEST"/>
-<wire x1="-2.54" y1="119.38" x2="-7.62" y2="119.38" width="0.1524" layer="91"/>
-<pinref part="SV1" gate="1" pin="4"/>
-<wire x1="-15.24" y1="118.11" x2="-7.62" y2="118.11" width="0.1524" layer="91"/>
-<wire x1="-7.62" y1="118.11" x2="-7.62" y2="119.38" width="0.1524" layer="91"/>
+<wire x1="-15.24" y1="118.11" x2="-3.81" y2="118.11" width="0.1524" layer="91"/>
+<wire x1="-3.81" y1="118.11" x2="-2.54" y2="119.38" width="0.1524" layer="91"/>
+<pinref part="JP3" gate="G$1" pin="4"/>
 </segment>
 </net>
@@
 <pinref part="IC1" gate="G$1" pin="RST"/>
 <wire x1="-15.24" y1="115.57" x2="-11.43" y2="115.57" width="0.1524" layer="91"/>
-<wire x1="-11.43" y1="115.57" x2="-2.54" y2="115.57" width="0.1524" layer="91"/>
-<wire x1="-2.54" y1="115.57" x2="-2.54" y2="114.3" width="0.1524" layer="91"/>
-<pinref part="SV1" gate="1" pin="3"/>
+<wire x1="-11.43" y1="115.57" x2="-3.81" y2="115.57" width="0.1524" layer="91"/>
+<wire x1="-3.81" y1="115.57" x2="-2.54" y2="114.3" width="0.1524" layer="91"/>
 <pinref part="C18" gate="G$1" pin="2"/>
 <pinref part="R10" gate="G$1" pin="1"/>
@@
 <junction x="-11.43" y="115.57"/>
 <wire x1="-11.43" y1="115.57" x2="-11.43" y2="120.65" width="0.1524" layer="91"/>
+<pinref part="JP3" gate="G$1" pin="3"/>
 </segment>
 </net>
@@
 </segment>
 </net>
+<net name="INT2" class="0">
+<segment>
+<pinref part="IC1" gate="G$1" pin="P3.4"/>
+<wire x1="66.04" y1="119.38" x2="72.39" y2="119.38" width="0.1524" layer="91"/>
+<label x="71.12" y="119.38" size="1.778" layer="95"/>
+</segment>
+<segment>
+<pinref part="U$4" gate="G$1" pin="INT1"/>
+<wire x1="222.25" y1="156.21" x2="214.63" y2="156.21" width="0.1524" layer="91"/>
+<label x="214.63" y="156.21" size="1.778" layer="95"/>
+</segment>
+</net>
+<net name="N$14" class="0">
+<segment>
+<wire x1="232.664" y1="145.796" x2="234.188" y2="148.082" width="0.1524" layer="91"/>
+</segment>
+</net>
+<net name="N$15" class="0">
+<segment>
+<pinref part="U1" gate="G$1" pin="CHG"/>
+<wire x1="109.22" y1="223.52" x2="109.22" y2="217.17" width="0.1524" layer="91"/>
+<pinref part="R11" gate="G$1" pin="1"/>
+</segment>
+</net>
+<net name="N$18" class="0">
+<segment>
+<pinref part="R11" gate="G$1" pin="2"/>
+<pinref part="LED3" gate="G$1" pin="C"/>
+</segment>
+</net>

Commit message: done some routing
Parts:
- added D1: (no value), diode:DIODE-SOD523
- added IC3: (no value), SparkFun:V_REG_TPS76433SOT23-5
- added Q2: MOSFET-PCHANNEL, SparkFun:MOSFET-PCHANNEL
- added R12: (no value), rcl:R-EU_R0402
- added U2: MAX1555, SparkFun:MAX1555
Connections:
- removed net N$1: C11.2, LED3.A, U1.USB, X2.VBUS
- new net N$19: LED3.C, U1.CHG
- new net N$20: D1.C, IC3.IN, Q2.D
- new net N$21: D1.A, Q2.G, R12.1, U2.USB
- new net N$22: R12.2
- new net N$27: Q2.S, U2.BATT
- net KEEPON: now also IC1.P1.2; no longer IC1.P1.4
- net N$15: now also LED3.A; no longer U1.CHG
- net N$18: now also C11.2, U1.USB, X2.VBUS; no longer LED3.C
- net N$25: no longer R4.2
- net SWITCHON: now also IC1.P1.1; no longer IC1.P1.3
Other:
- note added: "not needed depending on reg"
- moved on the sheet: LED3, R11, R4
Changed lines of the file:
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@@
 <part name="R11" library="rcl" deviceset="R-EU_" device="R0402"/>
 <part name="LED3" library="SparkFun" deviceset="LED" device="0603"/>
+<part name="U2" library="SparkFun" deviceset="MAX1555" device=""/>
+<part name="IC3" library="SparkFun" deviceset="V_REG_TPS76433" device="SOT23-5"/>
+<part name="D1" library="diode" deviceset="DIODE-" device="SOD523"/>
+<part name="Q2" library="SparkFun" deviceset="MOSFET-PCHANNEL" device=""/>
+<part name="R12" library="rcl" deviceset="R-EU_" device="R0402"/>
 </parts>
 <sheets>
@@
 <text x="232.664" y="144.018" size="1.778" layer="91">3</text>
 <text x="109.22" y="245.11" size="1.778" layer="91">what happens when charging?</text>
+<text x="158.75" y="201.93" size="1.778" layer="91">not needed depending on reg</text>
 </plain>
 <instances>
@@
 <instance part="C17" gate="G$1" x="255.27" y="153.67" rot="MR180"/>
 <instance part="GND28" gate="1" x="255.27" y="148.59" smashed="yes"/>
-<instance part="R4" gate="G$1" x="157.48" y="204.47" rot="R90"/>
-<instance part="GND43" gate="1" x="157.48" y="195.58" smashed="yes"/>
+<instance part="R4" gate="G$1" x="157.48" y="201.93" rot="R90"/>
+<instance part="GND43" gate="1" x="157.48" y="194.31" smashed="yes"/>
 <instance part="+3V4" gate="G$1" x="237.49" y="195.58"/>
 <instance part="+3V5" gate="G$1" x="242.57" y="195.58"/>
@@
 <instance part="+3V3" gate="G$1" x="-12.7" y="110.49" rot="R270"/>
 <instance part="JP3" gate="G$1" x="-20.32" y="113.03"/>
-<instance part="R11" gate="G$1" x="109.22" y="212.09" rot="R270"/>
-<instance part="LED3" gate="G$1" x="109.22" y="201.93" rot="R180"/>
+<instance part="R11" gate="G$1" x="109.22" y="207.01" rot="R270"/>
+<instance part="LED3" gate="G$1" x="109.22" y="214.63" rot="R180"/>
+<instance part="U2" gate="G$1" x="121.92" y="278.13"/>
+<instance part="IC3" gate="G$1" x="162.56" y="273.05"/>
+<instance part="D1" gate="G$1" x="128.27" y="303.53"/>
+<instance part="Q2" gate="G$1" x="137.16" y="294.64" rot="MR90"/>
+<instance part="R12" gate="G$1" x="138.43" y="267.97" rot="R270"/>
 </instances>
 <busses>
@@
 <pinref part="R4" gate="G$1" pin="1"/>
 <pinref part="GND43" gate="1" pin="GND"/>
-<wire x1="157.48" y1="198.12" x2="157.48" y2="199.39" width="0.1524" layer="91"/>
 </segment>
 <segment>
@@
 <pinref part="GND30" gate="1" pin="GND"/>
 <pinref part="JP3" gate="G$1" pin="2"/>
-</segment>
-</net>
-<net name="N$1" class="0">
-<segment>
-<pinref part="X2" gate="G$1" pin="VBUS"/>
-<wire x1="99.06" y1="227.33" x2="101.6" y2="227.33" width="0.1524" layer="91"/>
-<wire x1="101.6" y1="227.33" x2="105.41" y2="227.33" width="0.1524" layer="91"/>
-<wire x1="105.41" y1="227.33" x2="105.41" y2="228.6" width="0.1524" layer="91"/>
-<pinref part="U1" gate="G$1" pin="USB"/>
-<wire x1="105.41" y1="228.6" x2="109.22" y2="228.6" width="0.1524" layer="91"/>
-<pinref part="C11" gate="G$1" pin="2"/>
-<junction x="105.41" y="228.6"/>
-<pinref part="LED3" gate="G$1" pin="A"/>
-<wire x1="109.22" y1="199.39" x2="101.6" y2="199.39" width="0.1524" layer="91"/>
-<wire x1="101.6" y1="199.39" x2="101.6" y2="227.33" width="0.1524" layer="91"/>
-<junction x="101.6" y="227.33"/>
 </segment>
 </net>
@@
 </segment>
 <segment>
-<pinref part="IC1" gate="G$1" pin="P1.4"/>
-<wire x1="66.04" y1="165.1" x2="72.39" y2="165.1" width="0.1524" layer="91"/>
-<label x="71.12" y="165.1" size="1.778" layer="95"/>
+<pinref part="IC1" gate="G$1" pin="P1.2"/>
+<wire x1="66.04" y1="170.18" x2="73.66" y2="170.18" width="0.1524" layer="91"/>
+<label x="71.12" y="170.18" size="1.778" layer="95"/>
 </segment>
 </net>
@@
 <segment>
 <pinref part="D3" gate="G$1" pin="C"/>
-<pinref part="R4" gate="G$1" pin="2"/>
 <pinref part="D4" gate="G$1" pin="C"/>
-<junction x="157.48" y="209.55"/>
 <pinref part="D4" gate="G$1" pin="C"/>
 <wire x1="157.48" y1="209.55" x2="157.48" y2="214.63" width="0.1524" layer="91"/>
@@
 <wire x1="157.48" y1="223.52" x2="154.94" y2="223.52" width="0.1524" layer="91"/>
 <wire x1="154.94" y1="214.63" x2="154.94" y2="223.52" width="0.1524" layer="91"/>
+<junction x="157.48" y="209.55"/>
 </segment>
 </net>
@@
 </segment>
 <segment>
-<pinref part="IC1" gate="G$1" pin="P1.3"/>
-<wire x1="66.04" y1="167.64" x2="72.39" y2="167.64" width="0.1524" layer="91"/>
-<label x="71.12" y="167.64" size="1.778" layer="95"/>
+<pinref part="IC1" gate="G$1" pin="P1.1"/>
+<wire x1="66.04" y1="172.72" x2="72.39" y2="172.72" width="0.1524" layer="91"/>
+<label x="71.12" y="172.72" size="1.778" layer="95"/>
 </segment>
 </net>
@@
 <net name="N$15" class="0">
 <segment>
+<pinref part="LED3" gate="G$1" pin="A"/>
+<pinref part="R11" gate="G$1" pin="1"/>
+</segment>
+</net>
+<net name="N$18" class="0">
+<segment>
+<wire x1="101.6" y1="198.12" x2="109.22" y2="198.12" width="0.1524" layer="91"/>
+<wire x1="109.22" y1="198.12" x2="109.22" y2="201.93" width="0.1524" layer="91"/>
+<pinref part="R11" gate="G$1" pin="2"/>
+<pinref part="X2" gate="G$1" pin="VBUS"/>
+<wire x1="99.06" y1="227.33" x2="101.6" y2="227.33" width="0.1524" layer="91"/>
+<wire x1="101.6" y1="227.33" x2="105.41" y2="227.33" width="0.1524" layer="91"/>
+<wire x1="105.41" y1="227.33" x2="105.41" y2="228.6" width="0.1524" layer="91"/>
+<pinref part="U1" gate="G$1" pin="USB"/>
+<wire x1="105.41" y1="228.6" x2="109.22" y2="228.6" width="0.1524" layer="91"/>
+<pinref part="C11" gate="G$1" pin="2"/>
+<junction x="105.41" y="228.6"/>
+<wire x1="101.6" y1="198.12" x2="101.6" y2="227.33" width="0.1524" layer="91"/>
+<junction x="101.6" y="227.33"/>
+</segment>
+</net>
+<net name="N$19" class="0">
+<segment>
 <pinref part="U1" gate="G$1" pin="CHG"/>
-<wire x1="109.22" y1="223.52" x2="109.22" y2="217.17" width="0.1524" layer="91"/>
-<pinref part="R11" gate="G$1" pin="1"/>
-</segment>
-</net>
-<net name="N$18" class="0">
-<segment>
-<pinref part="R11" gate="G$1" pin="2"/>
 <pinref part="LED3" gate="G$1" pin="C"/>
-</segment>
-</net>
+<wire x1="109.22" y1="223.52" x2="109.22" y2="219.71" width="0.1524" layer="91"/>
+</segment>
+</net>
+<net name="N$20" class="0">
+<segment>
+<pinref part="D1" gate="G$1" pin="C"/>
+<wire x1="130.81" y1="303.53" x2="149.86" y2="303.53" width="0.1524" layer="91"/>
+<wire x1="149.86" y1="303.53" x2="149.86" y2="294.64" width="0.1524" layer="91"/>
+<pinref part="IC3" gate="G$1" pin="IN"/>
+<wire x1="149.86" y1="294.64" x2="149.86" y2="280.67" width="0.1524" layer="91"/>
+<wire x1="149.86" y1="280.67" x2="154.94" y2="280.67" width="0.1524" layer="91"/>
+<pinref part="Q2" gate="G$1" pin="D"/>
+<wire x1="142.24" y1="294.64" x2="149.86" y2="294.64" width="0.1524" layer="91"/>
+</segment>
+</net>
+<net name="N$21" class="0">
+<segment>
+<pinref part="Q2" gate="G$1" pin="G"/>
+<wire x1="137.16" y1="287.02" x2="138.43" y2="287.02" width="0.1524" layer="91"/>
+<wire x1="138.43" y1="287.02" x2="138.43" y2="273.05" width="0.1524" layer="91"/>
+<pinref part="R12" gate="G$1" pin="1"/>
+<pinref part="U2" gate="G$1" pin="USB"/>
+<wire x1="106.68" y1="280.67" x2="104.14" y2="280.67" width="0.1524" layer="91"/>
+<wire x1="104.14" y1="280.67" x2="95.25" y2="280.67" width="0.1524" layer="91"/>
+<wire x1="104.14" y1="280.67" x2="104.14" y2="303.53" width="0.1524" layer="91"/>
+<pinref part="D1" gate="G$1" pin="A"/>
+<wire x1="104.14" y1="303.53" x2="120.65" y2="303.53" width="0.1524" layer="91"/>
+<wire x1="120.65" y1="303.53" x2="125.73" y2="303.53" width="0.1524" layer="91"/>
+<wire x1="137.16" y1="287.02" x2="120.65" y2="287.02" width="0.1524" layer="91"/>
+<wire x1="120.65" y1="287.02" x2="120.65" y2="303.53" width="0.1524" layer="91"/>
+</segment>
+</net>
+<net name="N$22" class="0">
+<segment>
+<pinref part="R12" gate="G$1" pin="2"/>
+<wire x1="138.43" y1="262.89" x2="138.43" y2="260.35" width="0.1524" layer="91"/>
+<wire x1="138.43" y1="260.35" x2="137.16" y2="260.35" width="0.1524" layer="91"/>
+<wire x1="137.16" y1="260.35" x2="137.16" y2="259.08" width="0.1524" layer="91"/>
+<wire x1="137.16" y1="259.08" x2="139.7" y2="259.08" width="0.1524" layer="91"/>
+<wire x1="139.7" y1="259.08" x2="139.7" y2="260.35" width="0.1524" layer="91"/>
+</segment>
+</net>
+<net name="N$27" class="0">
+<segment>
+<pinref part="U2" gate="G$1" pin="BATT"/>
+<pinref part="Q2" gate="G$1" pin="S"/>
+<wire x1="134.62" y1="280.67" x2="132.08" y2="280.67" width="0.1524" layer="91"/>
+<wire x1="132.08" y1="280.67" x2="132.08" y2="294.64" width="0.1524" layer="91"/>
+</segment>
+</net>
